Commit message: add raft  simulator

File: src/omnibot_description/urdf/RTK.urdf.xacro (robot description, xacro)
@@ -1,4 +1,4 @@
 <?xml version="1.0"?>
-<robot name="omnibot" xmlns:xacro="http://www.ros.org/wiki/xacro">
+<robot name="omnibot_robot" xmlns:xacro="http://www.ros.org/wiki/xacro">
     <xacro:include filename="$(find omnibot_manipulator)/urdf/angle_arm.urdf"/>
     <xacro:include filename="$(find omnibot_platform)/urdf/platform.urdf.xacro"/>
@@ -6,5 +6,5 @@
         <parent link="base_link"/>
         <child link="ang_link0"/>
-        <origin xyz="0.0 0.1 0.04" rpy="0.0 0.0 3.14"/>
+        <origin xyz="0.0 0.096 0.113" rpy="0.0 0.0 3.14"/>
     </joint>
 </robot>

File: src/omnibot_platform/urdf/platform.urdf.xacro (robot description, xacro)
@@ -1,8 +1,8 @@
 <?xml version="1.0"?>
 <robot name="omnibot_platform" xmlns:xacro="http://www.ros.org/wiki/xacro">
-    <xacro:property name="base_lenth" value="0.265" />
-    <xacro:property name="base_width" value="0.385" />
+    <xacro:property name="base_lenth" value="0.30510" />
+    <xacro:property name="base_width" value="0.336" />
     <xacro:property name="base_height" value="0.15" />
-    <xacro:property name="wheel_x_offset" value="${(base_lenth / 2) + 0.03}" />
+    <xacro:property name="wheel_x_offset" value="${(base_lenth / 2)}" />
     <xacro:property name="wheel_y_offset" value="${(base_width / 2)}" />
     <!-- wheel template -->
@@ -10,5 +10,5 @@
         <link name="${suffix}_wheel_link">
             <visual name="">
-                <origin xyz="0.2 0.0 0.0" rpy="0.0 0.0 1.57" />
+                <origin xyz="0.0 0.0 0.0" rpy="0.0 0.0 0.0" />
                 <geometry>
                     <mesh filename="package://omnibot_platform/meshes/wheel.STL" scale="0.001 0.001 0.001" />
@@ -30,5 +30,5 @@
             <parent link="base_link" />
             <child link="${suffix}_wheel_link" />
-            <axis xyz="1.0 0.0 0.0" />
+            <axis xyz="0.0 0.0 1.0" />
             <limit effort="0.0" velocity="0.0" />
         </joint>
@@ -47,7 +47,7 @@
     <link name="base_link">
         <visual name="">
-            <origin xyz="0.0 0.0 0.0" rpy="0.0 0.0 0.0" />
+            <origin xyz="0.0 0.0 0.0" rpy="-1.57 0.0 3.14" />
             <geometry>
-                <box size="${base_lenth} ${base_width} ${base_height/2}" />
+                <mesh filename="package://omnibot_platform/meshes/base.STL" scale="0.001 0.001 0.001"/>
             </geometry>
             <material name="">
@@ -59,19 +59,19 @@
             <origin xyz="0.0 0.0 0.0" rpy="0.0 0.0 0.0" />
             <geometry>
-                <box size="${base_lenth} ${base_width} ${base_height/2}" />
+                <mesh filename="package://omnibot_platform/meshes/base.STL" scale="0.001 0.001 0.001"/>
             </geometry>
         </collision>
     </link>
     <xacro:wheel_template suffix="left_forward">
-        <origin xyz="${-wheel_x_offset} ${wheel_y_offset} 0.0" rpy="0.0 0.0 0.0" />
+        <origin xyz="${-wheel_x_offset} ${wheel_y_offset} 0.013285" rpy="0.0 1.57 0.0" />
     </xacro:wheel_template>
     <xacro:wheel_template suffix="right_forward">
-        <origin xyz="${wheel_x_offset} ${wheel_y_offset} 0.0" rpy="0.0 0.0 0.0" />
+        <origin xyz="${wheel_x_offset} ${wheel_y_offset} 0.013285" rpy="0.0 -1.57 0.0" />
     </xacro:wheel_template>
     <xacro:wheel_template suffix="left_backward">
-        <origin xyz="${-wheel_x_offset} ${-wheel_y_offset} 0.0" rpy="0.0 0.0 0.0" />
+        <origin xyz="${-wheel_x_offset} ${-wheel_y_offset} 0.013285" rpy="0.0 1.57 0.0" />
     </xacro:wheel_template>
     <xacro:wheel_template suffix="right_backward">
-        <origin xyz="${wheel_x_offset} ${-wheel_y_offset} 0.0" rpy="0.0 0.0 0.0" />
+        <origin xyz="${wheel_x_offset} ${-wheel_y_offset} 0.013285" rpy="0.0 -1.57 0.0" />
     </xacro:wheel_template>
 </robot>
