Commit message: add gazebo sim with controllers

File: src/omnibot_description/urdf/omnibot_robot.urdf (robot description, URDF)
Before this commit: robot omnibot_robot, 14 links, 13 joints
Links:
- link base_link: mass None -> 3.0; geometry collision mesh filename=package://omnibot_platform/meshes/hodovaya_low.dae scale=0.001 0.001 0.001; visual mesh filename=package://omnibot_platform/meshes/hodovaya_low.dae scale=0.001 0.001 0.001
- link left_backward_wheel_link: mass None -> 0.2; geometry collision mesh filename=package://omnibot_platform/meshes/wheel_low.dae scale=0.001 0.001 0.001; visual mesh filename=package://omnibot_platform/meshes/wheel_low.dae scale=0.001 0.001 0.001
- link left_forward_wheel_link: mass None -> 0.2; geometry collision mesh filename=package://omnibot_platform/meshes/wheel_low.dae scale=0.001 0.001 0.001; visual mesh filename=package://omnibot_platform/meshes/wheel_low.dae scale=0.001 0.001 0.001
- link right_backward_wheel_link: mass None -> 0.2; geometry collision mesh filename=package://omnibot_platform/meshes/wheel_low.dae scale=0.001 0.001 0.001; visual mesh filename=package://omnibot_platform/meshes/wheel_low.dae scale=0.001 0.001 0.001
- link right_forward_wheel_link: mass None -> 0.2; geometry collision mesh filename=package://omnibot_platform/meshes/wheel_low.dae scale=0.001 0.001 0.001; visual mesh filename=package://omnibot_platform/meshes/wheel_low.dae scale=0.001 0.001 0.001
- link tip_link: mass None -> 0.00002
Joints:
- joint left_backward_wheel_joint: axis 0.0 0.0 1.0 -> 0.0 1.0 0.0; origin xyz=-0.15255 -0.168 0.013285 rpy=0.0 1.57 0.0 -> xyz=-0.15255 -0.168 0.013285 rpy=0.0 0.0  1.57
- joint left_forward_wheel_joint: axis 0.0 0.0 1.0 -> 0.0 1.0 0.0; origin xyz=-0.15255 0.168 0.013285 rpy=0.0 1.57 0.0 -> xyz=-0.15255 0.168 0.013285 rpy=0.0 0.0 1.57
- joint right_backward_wheel_joint: axis 0.0 0.0 1.0 -> 0.0 1.0 0.0; origin xyz=0.15255 -0.168 0.013285 rpy=0.0 -1.57 0.0 -> xyz=0.15255 -0.168 0.013285 rpy=0.0 0.0  -1.57
- joint right_forward_wheel_joint: axis 0.0 0.0 1.0 -> 0.0 1.0 0.0; origin xyz=0.15255 0.168 0.013285 rpy=0.0 -1.57 0.0 -> xyz=0.15255 0.168 0.013285 rpy=0.0 0.0 -1.57

File: src/omnibot_description/urdf/omnibot_robot.urdf.xacro (robot description, xacro)
@@ -1,5 +1,11 @@
 <?xml version="1.0"?>
 <robot name="omnibot_robot" xmlns:xacro="http://www.ros.org/wiki/xacro">
-    <xacro:include filename="$(find omnibot_manipulator)/urdf/angle_arm.urdf"/>
+<gazebo>
+  <plugin name="gazebo_ros_control" filename="libgazebo_ros_control.so">
+    <!-- <robotNamespace>/omnibot_robot</robotNamespace> -->
+    <robotSimType>gazebo_ros_control/DefaultRobotHWSim</robotSimType>
+  </plugin>
+</gazebo>
+    <xacro:include filename="$(find omnibot_manipulator)/urdf/manipulator.urdf"/>
     <xacro:include filename="$(find omnibot_platform)/urdf/platform.urdf.xacro"/>
     <joint name="manip2platform_connector" type="fixed">

File: src/omnibot_manipulator/urdf/manipulator.urdf (robot description, URDF)
Before this commit: robot angle_robot, 9 links, 8 joints
Links:
- link tip_link: mass None -> 0.00002

File: src/omnibot_platform/urdf/platform.urdf.xacro (robot description, xacro)
@@ -24,4 +24,9 @@
                 </geometry>
             </collision>
+            <inertial>
+			    <origin xyz="0 0.0 0" rpy="0 0 0" />
+			    <mass value="0.2" />
+			    <inertia ixx="0.01" ixy="0.0" ixz="0.0" iyy="0.01" iyz="0.0" izz="0.01" />
+		    </inertial>
         </link>
         <joint name="${suffix}_wheel_joint" type="continuous">
@@ -29,5 +34,5 @@
             <parent link="base_link" />
             <child link="${suffix}_wheel_link" />
-            <axis xyz="0.0 0.0 1.0" />
+            <axis xyz="0.0 1.0 0.0" />
             <limit effort="0.0" velocity="0.0" />
         </joint>
@@ -35,5 +40,5 @@
             <type>transmission_interface/SimpleTransmission</type>
             <actuator name="${suffix}_wheel_motor">
-                <hardwareInterface>hardware_interface/VelocityJointInterface</hardwareInterface>
+                <hardwareInterface>hardware_interface/VelocityJointInterface </hardwareInterface>
                 <mechanicalReduction>1</mechanicalReduction>
             </actuator>
@@ -55,9 +60,14 @@
         </visual>
         <collision>
-            <origin xyz="0.0 0.0 0.0" rpy="0.0 0.0 0.0" />
+            <origin xyz="0.0 0.0 0.0" rpy="0.0 3.14 0.0"  />
             <geometry>
                 <mesh filename="package://omnibot_platform/meshes/hodovaya_low.dae" scale="0.001 0.001 0.001"/>
             </geometry>
         </collision>
+        <inertial>
+			<origin xyz="0 0.0 0" rpy="0 0 0" />
+			<mass value="3.0" />
+			<inertia ixx="1.0" ixy="1.0" ixz="1.0" iyy="0.01" iyz="0.0" izz="0.01" />
+		</inertial>
     </link>
     <xacro:wheel_template suffix="left_forward">
@@ -65,5 +75,5 @@
     </xacro:wheel_template>
     <xacro:wheel_template suffix="right_forward">
-        <origin xyz="${wheel_x_offset} ${wheel_y_offset} 0.013285" rpy="0.0 0.0 1.57" />
+        <origin xyz="${wheel_x_offset} ${wheel_y_offset} 0.013285" rpy="0.0 0.0 -1.57" />
     </xacro:wheel_template>
     <xacro:wheel_template suffix="left_backward">
@@ -71,5 +81,5 @@
     </xacro:wheel_template>
     <xacro:wheel_template suffix="right_backward">
-        <origin xyz="${wheel_x_offset} ${-wheel_y_offset} 0.013285" rpy="0.0 0.0  1.57" />
+        <origin xyz="${wheel_x_offset} ${-wheel_y_offset} 0.013285" rpy="0.0 0.0  -1.57" />
     </xacro:wheel_template>
 </robot>

Commit message: SYNS_FROM_ROBOT_PC

File: src/omnibot_description/urdf/omnibot_robot.urdf (robot description, URDF)
Before this commit: robot omnibot_robot, 14 links, 13 joints
Links:
- link base_link: mass 3.0 -> 5.0
- link left_backward_wheel_link: mass 0.2 -> 0.5
- link left_forward_wheel_link: mass 0.2 -> 0.5
- link right_backward_wheel_link: mass 0.2 -> 0.5
- link right_forward_wheel_link: mass 0.2 -> 0.5
Joints:
- joint left_backward_wheel_joint: limit effort=0.0 velocity=0.0 -> effort=5.0 velocity=100000.0
- joint left_forward_wheel_joint: limit effort=0.0 velocity=0.0 -> effort=5.0 velocity=100000.0
- joint right_backward_wheel_joint: limit effort=0.0 velocity=0.0 -> effort=5.0 velocity=100000.0
- joint right_forward_wheel_joint: limit effort=0.0 velocity=0.0 -> effort=5.0 velocity=100000.0

File: src/omnibot_description/urdf/omnibot_robot.urdf.xacro (robot description, xacro)
@@ -1,16 +1,24 @@
 <?xml version="1.0"?>
 <robot name="omnibot_robot" xmlns:xacro="http://www.ros.org/wiki/xacro">
-<gazebo>
-  <plugin name="gazebo_ros_control" filename="libgazebo_ros_control.so">
-    <!-- <robotNamespace>/omnibot_robot</robotNamespace> -->
-    <robotSimType>gazebo_ros_control/DefaultRobotHWSim</robotSimType>
-  </plugin>
-</gazebo>
-    <xacro:include filename="$(find omnibot_manipulator)/urdf/manipulator.urdf"/>
-    <xacro:include filename="$(find omnibot_platform)/urdf/platform.urdf.xacro"/>
-    <joint name="manip2platform_connector" type="fixed">
-        <parent link="base_link"/>
-        <child link="ang_link0"/>
-        <origin xyz="0.0 0.096 0.113" rpy="0.0 0.0 3.14"/>
-    </joint>
+  <gazebo>
+    <!-- <plugin name="gazebo_ros_control" filename="libgazebo_ros_planar_move.so"> -->
+      <plugin name="gazebo_ros_control" filename="libgazebo_ros_control.so">
+      <!-- <plugin name="differential_drive_controller" filename="libdiffdrive_plugin.so"> -->
+      <!-- <robotNamespace>/omnibot_robot</robotNamespace> -->
+      <robotSimType>gazebo_ros_control/DefaultRobotHWSim</robotSimType>
+      <!-- <commandTopic>cmd_vel</commandTopic> -->
+      <odometryTopic>odom</odometryTopic>
+      <odometryFrame>odom</odometryFrame>
+      <odometryRate>100.0</odometryRate>
+      <robotBaseFrame>base_footprint</robotBaseFrame>
+      <publishTF>false</publishTF>
+    </plugin>
+  </gazebo>
+  <xacro:include filename="$(find omnibot_manipulator)/urdf/manipulator.urdf" />
+  <xacro:include filename="$(find omnibot_platform)/urdf/platform.urdf.xacro" />
+  <joint name="manip2platform_connector" type="fixed">
+    <parent link="base_link" />
+    <child link="ang_link0" />
+    <origin xyz="0.0 0.096 0.113" rpy="0.0 0.0 3.14" />
+  </joint>
 </robot>

File: src/omnibot_platform/urdf/platform.urdf.xacro (robot description, xacro)
@@ -3,7 +3,30 @@
     <xacro:property name="base_lenth" value="0.30510" />
     <xacro:property name="base_width" value="0.336" />
-    <xacro:property name="base_height" value="0.15" />
+    <xacro:property name="base_height" value="0.200" />
+    <xacro:property name="robot_mass" value="5.0" />
+    <xacro:property name="wheel_mass" value="0.5" />
+    <xacro:property name="wheel_deameter" value="0.15" />
+    <xacro:property name="wheel_radius" value="${wheel_deameter/2}" />
+    <xacro:property name="wheel_width" value="0.3" />
     <xacro:property name="wheel_x_offset" value="${(base_lenth / 2)}" />
     <xacro:property name="wheel_y_offset" value="${(base_width / 2)}" />
+    <xacro:macro name="cylinder_inertia_calculator" params="*origin m r h">
+        <inertial>
+            <xacro:insert_block name="origin" />
+            <mass value="${m}" />
+            <!-- <inertia ixx="${m*(3*r*r+h*h)/12}" ixy="0" ixz="0" iyy="${m*(3*r*r+h*h)/12}" iyz="0" izz="${m*r*r/2}" /> -->
+            <!-- <inertia ixx="0.012411765597" ixy="-0.000711733678" ixz="0.00050272983" iyy="0.015218160428" iyz="-0.000004273467" izz="0.011763977943" /> -->
+           <!-- <inertia ixx="1e-10" ixy="0.0" ixz="1e-10" iyy="0.0" iyz="0.0" izz="1e-10"/> -->
+          <inertia ixx="0.0" ixy="0.0" ixz="0.0" iyy="0.0" iyz="0.0" izz="0.0"/>
+        </inertial>
+    </xacro:macro>
+    <xacro:macro name="box_inertia_calculator" params="*origin m x y z">
+        <inertial>
+            <xacro:insert_block name="origin" />
+            <mass value="${m}" />
+            <!-- <inertia ixx="${0.83*m*(y+z)}" ixy="0.0" ixz="0.0" iyy="${0.83*m*(x+z)}" iyz="0.0" izz="${0.83*m*(y+x)}" /> -->
+            <inertia ixx="0.0" ixy="0.0" ixz="0.0" iyy="0.0" iyz="0.0" izz="0.0"/>
+        </inertial>
+    </xacro:macro>
     <xacro:macro name="wheel_template" params="suffix *origin">
         <link name="${suffix}_wheel_link">
@@ -24,10 +47,16 @@
                 </geometry>
             </collision>
-            <inertial>
-			    <origin xyz="0 0.0 0" rpy="0 0 0" />
-			    <mass value="0.2" />
-			    <inertia ixx="0.01" ixy="0.0" ixz="0.0" iyy="0.01" iyz="0.0" izz="0.01" />
-		    </inertial>
+            <xacro:cylinder_inertia_calculator m="${wheel_mass}" r="${wheel_radius}" h="${wheel_width}">
+                <xacro:insert_block name="origin" />
+            </xacro:cylinder_inertia_calculator>
         </link>
+        <gazebo reference="${suffix}_wheel_link">
+            <kp>10000.0</kp>
+            <kd>10000.0</kd>
+            <mu1>1000.0</mu1>
+            <mu2>1000.0</mu2>
+            <minDepth>0.001</minDepth>
+            <maxVel>1.0</maxVel>
+        </gazebo>
         <joint name="${suffix}_wheel_joint" type="continuous">
             <xacro:insert_block name="origin" />
@@ -35,5 +64,5 @@
             <child link="${suffix}_wheel_link" />
             <axis xyz="0.0 1.0 0.0" />
-            <limit effort="0.0" velocity="0.0" />
+            <limit effort="5.0" velocity="100000.0" />
         </joint>
         <transmission name="${suffix}_wheel_transmission" type="SimpleTransmission">
@@ -52,5 +81,5 @@
             <origin xyz="0.0 0.0 0.0" rpy="0.0 3.14 0.0" />
             <geometry>
-                <mesh filename="package://omnibot_platform/meshes/hodovaya_low.dae" scale="0.001 0.001 0.001"/>
+                <mesh filename="package://omnibot_platform/meshes/hodovaya_low.dae" scale="0.001 0.001 0.001" />
             </geometry>
             <material name="">
@@ -60,14 +89,12 @@
         </visual>
         <collision>
-            <origin xyz="0.0 0.0 0.0" rpy="0.0 3.14 0.0"  />
+            <origin xyz="0.0 0.0 0.0" rpy="0.0 3.14 0.0" />
             <geometry>
-                <mesh filename="package://omnibot_platform/meshes/hodovaya_low.dae" scale="0.001 0.001 0.001"/>
+                <mesh filename="package://omnibot_platform/meshes/hodovaya_low.dae" scale="0.001 0.001 0.001" />
             </geometry>
         </collision>
-        <inertial>
-			<origin xyz="0 0.0 0" rpy="0 0 0" />
-			<mass value="3.0" />
-			<inertia ixx="1.0" ixy="1.0" ixz="1.0" iyy="0.01" iyz="0.0" izz="0.01" />
-		</inertial>
+        <xacro:box_inertia_calculator m="${robot_mass}" x="${base_lenth}" y="${base_width}" z="${base_height}">
+            <origin xyz="0.0 0.0 0.0" rpy="0.0 3.14 0.0" />
+        </xacro:box_inertia_calculator>
     </link>
     <xacro:wheel_template suffix="left_forward">
