Commit message: fix sync manipulator movements gazebo and rviz bug

File: src/omnibot_description/urdf/omnibot_description.urdf.xacro (robot description, xacro)
@@ -7,7 +7,7 @@
     <xacro:include filename="$(find omnibot_manipulator_description)/urdf/omnibot_manipulator.urdf.xacro"/>
     <joint name="manipulator_connector" type="fixed">
-        <parent link="base_link" />
+        <parent link="base_footprint" />
         <child link="ang_link0" />
-        <origin xyz="0.096 0.0  0.113" rpy="0.0 0.0 0.0" />
+        <origin xyz="0.096 0.0  0.113" rpy="0.0 0.0 1.57" />
     </joint>
     </xacro:if>

File: src/omnibot_manipulator/omnibot_manipulator_description/urdf/omnibot_manipulator.urdf.xacro (robot description, xacro)
@@ -27,12 +27,12 @@
 	<xacro:property name="joint_5_upper_limit" value="2.60" />
 	<xacro:property name="joint_5_lower_limit" value="-2.60" />
-	<arg name="work_mode" default="notest"/>
-	<xacro:property name="mode" value="$(arg work_mode)"/>
+	<arg name="work_mode" default="notest" />
+	<xacro:property name="mode" value="$(arg work_mode)" />
 	<xacro:if value="${mode == 'test'}">
-		<link name="world"/>
+		<link name="world" />
 		<joint name="map2base" type="fixed">
-			<parent link="world"/>
-			<child link="ang_link0"/>
-			<origin xyz="0.0 0.0 0.0" rpy="0.0 0.0 0.0"/>
+			<parent link="world" />
+			<child link="ang_link0" />
+			<origin xyz="0.0 0.0 0.0" rpy="0.0 0.0 0.0" />
 		</joint>
 	</xacro:if>
@@ -46,5 +46,5 @@
 		<inertial>
 			<origin xyz="0 0 0.5" rpy="0 0 0" />
-			<mass value="1" />
+			<mass value="0.5" />
 			<inertia
 				ixx="0.01" ixy="0.0" ixz="0.0"
@@ -77,5 +77,5 @@
 		<inertial>
 			<origin xyz="0 0.25 0" rpy="0 0 0" />
-			<mass value="0.001" />
+			<mass value="0.3" />
 			<inertia
 				ixx="0.01" ixy="0.0" ixz="0.0"
@@ -107,5 +107,5 @@
 		<inertial>
 			<origin xyz="0 0.15 0" rpy="0 0 0" />
-			<mass value="0.001" />
+			<mass value="0.3" />
 			<inertia
 				ixx="0.01" ixy="0.0" ixz="0.0"
@@ -138,5 +138,5 @@
 		<inertial>
 			<origin xyz="0 0 0" rpy="0 0 0" />
-			<mass value="0.001" />
+			<mass value="0.3" />
 			<inertia
 				ixx="0.01" ixy="0.0" ixz="0.0"
@@ -169,5 +169,5 @@
 		<inertial>
 			<origin xyz="0 0 0" rpy="0 0 0" />
-			<mass value="0.001" />
+			<mass value="0.3" />
 			<inertia
 				ixx="0.01" ixy="0.0" ixz="0.0"
@@ -200,5 +200,5 @@
 		<inertial>
 			<origin xyz="0 0 0" rpy="0 0 0" />
-			<mass value="0.001" />
+			<mass value="0.3" />
 			<inertia
 				ixx="0.01" ixy="0.0" ixz="0.0"
@@ -236,5 +236,5 @@
 		<inertial>
 			<origin xyz="0 0 0" rpy="0 0 0" />
-			<mass value="0.001" />
+			<mass value="0.3" />
 			<inertia
 				ixx="0.01" ixy="0.0" ixz="0.0"
@@ -267,5 +267,5 @@
 		<inertial>
 			<origin xyz="0 0 0" rpy="0 0 0" />
-			<mass value="0.001" />
+			<mass value="0.1" />
 			<inertia
 				ixx="0.01" ixy="0.0" ixz="0.0"

File: src/omnibot_platform/omnibot_platform_description/urdf/wheel.xacro (robot description, xacro)
@@ -18,5 +18,5 @@
         <origin xyz="0 0 0" rpy="0 0 0" />
         <mass value="0.25"/>
-        <inertia ixx="0.00031" ixy="0" ixz="0" iyy="0.0005" iyz="0" izz="0.00031"/>
+        <inertia ixx="0.0031" ixy="0" ixz="0" iyy="0.005" iyz="0" izz="0.0031"/>
       </inertial>
     </link>

Commit message: cosmetical edit

File: src/omnibot_description/urdf/omnibot_description.urdf.xacro (robot description, xacro)
@@ -4,5 +4,5 @@
     <xacro:include filename="$(find omnibot_platform_description)/urdf/omnibot_platform.urdf.xacro" />
     <xacro:if value="$(arg use_manipulator)">
-        <xacro:arg name="work_mode" default="notest" />
+        <xacro:arg name="standalone_load" default="false" />
     <xacro:include filename="$(find omnibot_manipulator_description)/urdf/omnibot_manipulator.urdf.xacro"/>
     <joint name="manipulator_connector" type="fixed">

File: src/omnibot_manipulator/omnibot_manipulator_description/urdf/omnibot_manipulator.urdf.xacro (robot description, xacro)
@@ -1,4 +1,10 @@
 <?xml version="1.0"?>
 <robot name="omnibot_manipulator" xmlns:xacro="http://www.ros.org/wiki/xacro">
+	<arg name="standalone_load" default="true" />
+	<gazebo>
+		<plugin name="gazebo_ros_control" filename="libgazebo_ros_control.so">
+			<robotNamespace>/omnibot_manipulator</robotNamespace>
+		</plugin>
+	</gazebo>
 	<xacro:include
 		filename="$(find omnibot_manipulator_description)/urdf/omnibot_manipulator.gazebo" />
@@ -27,7 +33,5 @@
 	<xacro:property name="joint_5_upper_limit" value="2.60" />
 	<xacro:property name="joint_5_lower_limit" value="-2.60" />
-	<arg name="work_mode" default="notest" />
-	<xacro:property name="mode" value="$(arg work_mode)" />
-	<xacro:if value="${mode == 'test'}">
+	<xacro:if value="$(arg standalone_load)">
 		<link name="world" />
 		<joint name="map2base" type="fixed">

Commit message: cosmetic 2

File: src/omnibot_description/urdf/omnibot_description.urdf.xacro (robot description, xacro)
@@ -1,14 +1,22 @@
 <?xml version="1.0"?>
 <robot xmlns:xacro="http://www.ros.org/wiki/xacro" name="omnibot_robot">
-    <xacro:arg name="use_manipulator" default="false"/>
+    <xacro:arg name="use_manipulator" default="false" />
+    <xacro:arg name="robot_namespace" default="omnibot_robot" />
+    <xacro:arg name="standalone_load" default="false" />
+    <xacro:property name="ns" value="$(arg robot_namespace)"/>
+    <gazebo>
+        <plugin name="gazebo_ros_control" filename="libgazebo_ros_control.so">
+            <robotNamespace>${ns}</robotNamespace>
+        </plugin>
+    </gazebo>
     <xacro:include filename="$(find omnibot_platform_description)/urdf/omnibot_platform.urdf.xacro" />
     <xacro:if value="$(arg use_manipulator)">
-        <xacro:arg name="standalone_load" default="false" />
-    <xacro:include filename="$(find omnibot_manipulator_description)/urdf/omnibot_manipulator.urdf.xacro"/>
-    <joint name="manipulator_connector" type="fixed">
-        <parent link="base_footprint" />
-        <child link="ang_link0" />
-        <origin xyz="0.096 0.0  0.113" rpy="0.0 0.0 1.57" />
-    </joint>
+        <xacro:include
+            filename="$(find omnibot_manipulator_description)/urdf/omnibot_manipulator.urdf.xacro" />
+        <joint name="manipulator_connector" type="fixed">
+            <parent link="base_footprint" />
+            <child link="ang_link0" />
+            <origin xyz="0.096 0.0  0.113" rpy="0.0 0.0 1.57" />
+        </joint>
     </xacro:if>
 </robot>

File: src/omnibot_manipulator/omnibot_manipulator_description/urdf/omnibot_manipulator.urdf.xacro (robot description, xacro)
@@ -2,9 +2,13 @@
 <robot name="omnibot_manipulator" xmlns:xacro="http://www.ros.org/wiki/xacro">
 	<arg name="standalone_load" default="true" />
-	<gazebo>
-		<plugin name="gazebo_ros_control" filename="libgazebo_ros_control.so">
-			<robotNamespace>/omnibot_manipulator</robotNamespace>
-		</plugin>
-	</gazebo>
+	<arg name="robot_namespace" default="omnibot_manipulator" />
+	<xacro:property name="ns" value="$(arg robot_namespace)" />
+	<xacro:unless value="${ns == '/' or ns != 'omnibot_manipulator'}">
+		<gazebo>
+			<plugin name="gazebo_ros_control" filename="libgazebo_ros_control.so">
+				<robotNamespace>${ns}</robotNamespace>
+			</plugin>
+		</gazebo>
+	</xacro:unless>
 	<xacro:include
 		filename="$(find omnibot_manipulator_description)/urdf/omnibot_manipulator.gazebo" />

File: src/omnibot_platform/omnibot_platform_description/urdf/omnibot_platform.urdf.xacro (robot description, xacro)
@@ -1,9 +1,13 @@
 <?xml version="1.0"?>
 <robot xmlns:xacro="http://www.ros.org/wiki/xacro" name="omnibot_platform">
+    <arg name="robot_namespace" default="omnibot_platform"/>
+    <xacro:property name="ns" value="$(arg robot_namespace)"/>
+    <xacro:unless value="${ns == '/' or ns != 'omnibot_manipulator'}">
     <gazebo>
         <plugin name="gazebo_ros_control" filename="libgazebo_ros_control.so">
-            <robotNamespace>/omnibot_platform</robotNamespace>
+            <robotNamespace>${ns}</robotNamespace>
         </plugin>
     </gazebo>
+</xacro:unless>
     <!-- BASELINK  -->
     <xacro:property name="wheel_base_width" value="0.306100" />

Commit message: add rs_d435, add sim start script, fix gazebo launch file

File: src/omnibot_description/urdf/omnibot_description.urdf.xacro (robot description, xacro)
@@ -4,7 +4,14 @@
     <xacro:arg name="robot_namespace" default="omnibot_robot" />
     <xacro:property name="ns" value="$(arg robot_namespace)"/>
+    <!-- <ros2_control name="GazeboSystem" type="system">
+    <hardware>
+        <plugin>gazebo_ros2_control/GazeboSystem</plugin>
+    </hardware>
+    <ros2_control> -->
     <gazebo>
-        <plugin name="gazebo_ros_control" filename="libgazebo_ros_control.so">
+        <plugin filename="libgazebo_ros2_control.so" name="gazebo_ros2_control">
             <robotNamespace>${ns}</robotNamespace>
+            <robot_sim_type>gazebo_ros2_control/GazeboSystem</robot_sim_type>
+             <parameters>$(find omnibot_gazebo)/config/controller_manager.yaml</parameters>
         </plugin>
     </gazebo>

File: src/omnibot_platform/omnibot_platform_description/urdf/_d435.urdf.xacro (robot description, xacro)
@@ -11,5 +11,5 @@
 <robot name="sensor_d435" xmlns:xacro="http://ros.org/wiki/xacro">
   <!--File includes-->
-  <xacro:include filename="$(find omnibot_platform_description)/urdf/_d435.gazebo.xacro"/>
+  <xacro:include filename="_d435.gazebo.xacro"/>
   <xacro:macro name="sensor_d435" params="parent
                                           name:=camera
@@ -67,5 +67,5 @@
         <geometry>
           <!-- <box size="${d435_cam_width} ${d435_cam_height} ${d435_cam_depth}"/> -->
-          <mesh filename="package://realsense2_description/meshes/d435.dae"/>
+          <mesh filename="file://$(find omnibot_platform_description)/meshes/d435.dae"/>
           <!--<mesh filename="package://realsense2_description/meshes/d435/d435.dae"/>-->
         </geometry>

File: src/omnibot_platform/omnibot_platform_description/urdf/omnibot_platform.urdf.xacro (robot description, xacro)
@@ -5,5 +5,5 @@
     <xacro:unless value="${ns == '/' or ns != 'omnibot_manipulator'}">
     <gazebo>
-        <plugin name="gazebo_ros_control" filename="libgazebo_ros_control.so">
+        <plugin filename="libgazebo_ros2_control.so" name="gazebo_ros2_control">
             <robotNamespace>${ns}</robotNamespace>
         </plugin>
@@ -19,6 +19,5 @@
     <xacro:property name="base_link_rotate_y" value="3.14" />
     <xacro:property name="base_link_rotate_z" value="-1.57" />
-    <xacro:property name="base_link_mesh_path"
-        value="file://$(find omnibot_platform_description)/meshes/ros_base_link.dae" />
+    <xacro:property name="base_link_mesh_path" value="file://$(find omnibot_platform_description)/meshes/ros_base_link.dae" />
     <xacro:property name="base_link_mesh_scale_x" value="0.001" />
     <xacro:property name="base_link_mesh_scale_y" value="0.001" />
@@ -28,11 +27,8 @@
     <xacro:property name="omniwheel_offset_y" value="${(wheel_base_width / 2) + 0.035}" />
     <xacro:property name="omniwheel_offset_z" value="0.015500" />
-    <xacro:property name="omniwheel_macro_path"
-        value="$(find omnibot_platform_description)/urdf/mecanum_wheel_macro.xacro" />
+    <xacro:property name="omniwheel_macro_path" value="$(find omnibot_platform_description)/urdf/mecanum_wheel_macro.xacro" />
     <!-- REALSENSE -->
-    <xacro:property name="t265_xacro_path"
-        value="$(find omnibot_platform_description)/urdf/_t265.urdf.xacro" />
-    <xacro:property name="d435_xacro_path"
-        value="$(find omnibot_platform_description)/urdf/_d435.urdf.xacro" />
+    <xacro:property name="t265_xacro_path" value="$(find omnibot_platform_description)/urdf/_t265.urdf.xacro" />
+    <xacro:property name="d435_xacro_path" value="$(find omnibot_platform_description)/urdf/_d435.urdf.xacro" />
     <xacro:property name="t265_x_offset" value="${0.191250 + 0.0135}" />
     <xacro:property name="t265_y_offset" value="0.0" />
@@ -48,6 +44,5 @@
     <xacro:property name="d435_z_rotate" value="0.0" />
     <!-- LIDAR -->
-    <xacro:property name="rplidar_a3_xacro_path"
-        value="$(find omnibot_platform_description)/urdf/rplidar_a3.urdf.xacro" />
+    <xacro:property name="rplidar_a3_xacro_path" value="$(find omnibot_platform_description)/urdf/rplidar_a3.urdf.xacro" />
     <xacro:property name="rplidar_a3_x_offset" value="0.168000"/>
     <xacro:property name="rplidar_a3_y_offset" value="0.0"/>
@@ -120,10 +115,10 @@
     </xacro:mecanum_wheel>
     <!-- <xacro:sensor_t265 parent="base_link" name="t265" topics_ns="t265"
-        odom_xyz="0.0 0.0 0.0" odom_rpy="0.0 0.0 0.0" unite_imu_method="true">
+        odom_xyz="0.0 0.0 0.0" odom_rpy="0.0 0.0 0.0" unite_imu_method ="true">
         <origin xyz="${t265_x_offset}  ${t265_y_offset} ${t265_z_offset}" rpy="${t265_x_rotate}  ${t265_y_rotate} ${t265_z_rotate}" />
-    </xacro:sensor_t265>
+    </xacro:sensor_t265> -->
     <xacro:sensor_d435 parent="base_link" name="d435" topics_ns="d435" align_depth="true" enable_pointCloud="true">
         <origin xyz="${d435_x_offset} ${d435_y_offset}  ${d435_z_offset}" rpy="${d435_x_rotate} ${d435_y_rotate}  ${d435_z_rotate}" />
-    </xacro:sensor_d435> -->
+    </xacro:sensor_d435>
     <xacro:rplidar_a3 suffix="front">
         <origin xyz="${rplidar_a3_x_offset} ${rplidar_a3_y_offset} ${rplidar_a3_z_offset}" rpy="${rplidar_a3_x_rotate} ${rplidar_a3_y_rotate} ${rplidar_a3_z_rotate}"/>
