Commit message: add t265

File: src/omnibot_description/urdf/omnibot_description.urdf.xacro (robot description, xacro)
@@ -4,14 +4,9 @@
     <xacro:arg name="robot_namespace" default="omnibot_robot" />
     <xacro:property name="ns" value="$(arg robot_namespace)"/>
-    <!-- <ros2_control name="GazeboSystem" type="system">
-    <hardware>
-        <plugin>gazebo_ros2_control/GazeboSystem</plugin>
-    </hardware>
-    <ros2_control> -->
     <gazebo>
         <plugin filename="libgazebo_ros2_control.so" name="gazebo_ros2_control">
             <robotNamespace>${ns}</robotNamespace>
             <robot_sim_type>gazebo_ros2_control/GazeboSystem</robot_sim_type>
-             <parameters>$(find omnibot_gazebo)/config/controller_manager.yaml</parameters>
+             <!-- <parameters>$(find omnibot_gazebo)/config/controller_manager.yaml</parameters> -->
         </plugin>
     </gazebo>

File: src/omnibot_platform/omnibot_platform_description/urdf/_t265.gazebo.xacro (robot description, xacro)
@@ -1,11 +1,3 @@
 <?xml version="1.0"?>
-<!--
-Aknolegment: This file was copied from the realsense repository of
-pal-robotics-forks( https://github.com/pal-robotics-forks/realsense/ )
-and modified to add IMU and odometry.
-License: Apache 2.0. See LICENSE file in root directory.
-Copyright(c) 2017 PAL Robotics, S.L. All Rights Reserved
-This is the Gazebo URDF model for the Intel RealSense T265 camera
--->
 <robot xmlns:xacro="http://ros.org/wiki/xacro">
   <xacro:macro name="gazebo_t265" params="camera_name topics_ns
@@ -42,5 +34,5 @@
       <!--<max_vel>0.01</max_vel>
       <min_depth>0</min_depth>-->
-      <sensor name="${camera_name}fisheye1" type="wideanglecamera">
+      <sensor name="${camera_name}_fisheye1" type="wideanglecamera">
         <!-- <origin xyz="0 0 0" rpy="0 ${M_PI/2} 0"/> -->
         <update_rate>${fisheye_fps}</update_rate>
@@ -68,5 +60,5 @@
           </lens>
         </camera>
-        <plugin name="${camera_name}fisheye1" filename="libgazebo_ros_camera.so">
+        <plugin name="${camera_name}_fisheye1" filename="libgazebo_ros_camera.so">
           <alwaysOn>true</alwaysOn>
           <updateRate>${fisheye_fps}</updateRate>
@@ -101,5 +93,5 @@
       <!--<max_vel>0.01</max_vel>
       <min_depth>0</min_depth>-->
-      <sensor name="${camera_name}fisheye2" type="wideanglecamera">
+      <sensor name="${camera_name}_fisheye2" type="wideanglecamera">
         <!-- <origin xyz="0 0 0" rpy="0 ${M_PI/2} 0"/> -->
         <update_rate>${fisheye_fps}</update_rate>
@@ -128,5 +120,5 @@
         </camera>
         <always_on>1</always_on>
-        <plugin name="${camera_name}fisheye2" filename="libgazebo_ros_camera.so">
+        <plugin name="${camera_name}_fisheye2" filename="libgazebo_ros_camera.so">
           <alwaysOn>true</alwaysOn>
           <updateRate>${fisheye_fps}</updateRate>
@@ -144,10 +136,11 @@
       </sensor>
       <!-- IMU -->
-      <xacro:if value="${unite_imu_method == 'copy' or unite_imu_method == 'linear_interpolation'}">
+      <!-- <xacro:if value="${unite_imu_method == 'copy' or unite_imu_method == 'linear_interpolation'}"> -->
         <sensor name="${camera_name}_imu" type="imu">
           <always_on>true</always_on>
           <update_rate>${gyro_fps}</update_rate>
           <topic>${camera_name}/imu/sample</topic>
-          <plugin name="{camera_name}imu" filename="libgazebo_ros_imu_sensor.so">
+          <plugin name="${camera_name}_imu" filename="libgazebo_ros_imu_sensor.so">
+            <initial_orientation_as_reference>false</initial_orientation_as_reference>
             <topicName>${camera_name}/imu/sample</topicName>
             <bodyName>${camera_name}_pose_frame</bodyName>
@@ -159,8 +152,8 @@
           </plugin>
         </sensor>
-      </xacro:if>
+      <!-- </xacro:if> -->
       <!-- Accel and gyro -->
       <xacro:unless value="${unite_imu_method == 'copy' or unite_imu_method == 'linear_interpolation'}">
-        <sensor name="{camera_name}accel" type="imu">
+        <sensor name="${camera_name}_accel" type="imu">
           <always_on>true</always_on>
           <update_rate>${accel_fps}</update_rate>
@@ -196,13 +189,20 @@
     <gazebo>
       <!-- Odom from SLAM -->
-      <plugin name="p3d_base_controller" filename="libgazebo_ros_p3d.so">
+      <plugin name="libgazebo_ros_p3d" filename="libgazebo_ros_p3d.so">
             <alwaysOn>true</alwaysOn>
             <updateRate>${odom_fps}</updateRate>
-            <bodyName>${pose_frame}</bodyName>
+            <bodyName>${camera_name}_pose_frame</bodyName>
             <topicName>${topics_ns}/odom/sample</topicName>
             <gaussianNoise>0.01</gaussianNoise>
-            <frameName>map</frameName>
             <xyzOffsets>${odom_xyz}</xyzOffsets>
             <rpyOffsets>${odom_rpy}</rpyOffsets>
+            <ros>
+              <namespace>t265</namespace>
+              <remapping>odom:=odom</remapping>
+              </ros>
+              <frame_name>map</frame_name>
+              <body_name>base_footprint</body_name>
+              <update_rate>200.0</update_rate>
+              <gaussian_noise>0.01</gaussian_noise>
         </plugin>
     </gazebo>

File: src/omnibot_platform/omnibot_platform_description/urdf/_t265.urdf.xacro (robot description, xacro)
@@ -12,5 +12,5 @@
 <robot name="sensor_t265" xmlns:xacro="http://ros.org/wiki/xacro">
   <!--File includes-->
-  <xacro:include filename="$(find omnibot_platform_description)/urdf/_t265.gazebo.xacro"/>
+  <xacro:include filename="_t265.gazebo.xacro"/>
     <!-- odom_xyz, odom_rpy params are the transformation from the robot base_link to the camera reference frame (camerea_pose_frame)
   they are needed for the simulation of the camera slam capabilities -->
@@ -50,5 +50,5 @@
       <origin xyz="0 0 0" rpy="${M_PI / 2} 0 ${M_PI /2}"/>
         <geometry>
-            <mesh filename="package://omnibot_platform_description/meshes/t265_full.stl" scale="0.001 0.001 0.001"/>
+            <mesh filename="file://$(find omnibot_platform_description)/meshes/t265_full.stl" scale="0.001 0.001 0.001"/>
         </geometry>
         <material name="${name}_aluminum"/>
@@ -57,5 +57,5 @@
         <origin xyz="0 0 0" rpy="${M_PI / 2} 0 ${M_PI /2}"/>
         <geometry>
-          <mesh filename="package://omnibot_platform_description/meshes/t265_simplified.stl"  scale="0.001 0.001 0.001"/>
+          <mesh filename="file://$(find omnibot_platform_description)/meshes/t265_simplified.stl"  scale="0.001 0.001 0.001"/>
         </geometry>
       </collision>

File: src/omnibot_platform/omnibot_platform_description/urdf/mecanum_wheel_macro.xacro (robot description, xacro)
@@ -1,6 +1,6 @@
 <?xml version="1.0" ?>
 <robot name="mecanum_wheel" xmlns:xacro="http://ros.org/wiki/xacro">
-  <xacro:include filename="$(find omnibot_platform_description)/urdf/wheel.xacro" />
-  <xacro:include filename="$(find omnibot_platform_description)/urdf/rollers.xacro"  />
+  <xacro:include filename="wheel.xacro" />
+  <xacro:include filename="rollers.xacro"  />
   <xacro:macro name="mecanum_wheel" params="name side interface *origin parent">
     <xacro:wheel_link name="${name}" side="${side}" />

File: src/omnibot_platform/omnibot_platform_description/urdf/omnibot_platform.urdf.xacro (robot description, xacro)
@@ -4,10 +4,10 @@
     <xacro:property name="ns" value="$(arg robot_namespace)"/>
     <xacro:unless value="${ns == '/' or ns != 'omnibot_manipulator'}">
-    <gazebo>
-        <plugin filename="libgazebo_ros2_control.so" name="gazebo_ros2_control">
-            <robotNamespace>${ns}</robotNamespace>
-        </plugin>
-    </gazebo>
-</xacro:unless>
+        <gazebo>
+            <plugin filename="libgazebo_ros2_control.so" name="gazebo_ros2_control">
+                <robotNamespace>${ns}</robotNamespace>
+            </plugin>
+        </gazebo>
+    </xacro:unless>
     <!-- BASELINK  -->
     <xacro:property name="wheel_base_width" value="0.306100" />
@@ -27,8 +27,8 @@
     <xacro:property name="omniwheel_offset_y" value="${(wheel_base_width / 2) + 0.035}" />
     <xacro:property name="omniwheel_offset_z" value="0.015500" />
-    <xacro:property name="omniwheel_macro_path" value="$(find omnibot_platform_description)/urdf/mecanum_wheel_macro.xacro" />
+    <xacro:property name="omniwheel_macro_path" value="mecanum_wheel_macro.xacro" />
     <!-- REALSENSE -->
-    <xacro:property name="t265_xacro_path" value="$(find omnibot_platform_description)/urdf/_t265.urdf.xacro" />
-    <xacro:property name="d435_xacro_path" value="$(find omnibot_platform_description)/urdf/_d435.urdf.xacro" />
+    <xacro:property name="t265_xacro_path" value="_t265.urdf.xacro" />
+    <xacro:property name="d435_xacro_path" value="_d435.urdf.xacro" />
     <xacro:property name="t265_x_offset" value="${0.191250 + 0.0135}" />
     <xacro:property name="t265_y_offset" value="0.0" />
@@ -44,5 +44,5 @@
     <xacro:property name="d435_z_rotate" value="0.0" />
     <!-- LIDAR -->
-    <xacro:property name="rplidar_a3_xacro_path" value="$(find omnibot_platform_description)/urdf/rplidar_a3.urdf.xacro" />
+    <xacro:property name="rplidar_a3_xacro_path" value="rplidar_a3.urdf.xacro" />
     <xacro:property name="rplidar_a3_x_offset" value="0.168000"/>
     <xacro:property name="rplidar_a3_y_offset" value="0.0"/>
@@ -61,8 +61,6 @@
     <link name="base_link">
         <inertial>
-            <origin xyz="${base_link_offset_x} ${base_link_offset_y}
-        ${base_link_offset_z}"
-                rpy="${base_link_rotate_x} ${base_link_rotate_y}
-        ${base_link_rotate_z}" />
+            <origin xyz="${base_link_offset_x} ${base_link_offset_y} ${base_link_offset_z}"
+                rpy="${base_link_rotate_x} ${base_link_rotate_y} ${base_link_rotate_z}" />
             <mass value="3.0" />
             <xacro:box_inertia m="3.0" x="${wheel_base_width}" y="${wheel_base_lenth}" z="0.2" />
@@ -114,8 +112,9 @@
             rpy="0.0 0.0 -1.57" />
     </xacro:mecanum_wheel>
-    <!-- <xacro:sensor_t265 parent="base_link" name="t265" topics_ns="t265"
-        odom_xyz="0.0 0.0 0.0" odom_rpy="0.0 0.0 0.0" unite_imu_method ="true">
-        <origin xyz="${t265_x_offset}  ${t265_y_offset} ${t265_z_offset}" rpy="${t265_x_rotate}  ${t265_y_rotate} ${t265_z_rotate}" />
-    </xacro:sensor_t265> -->
+    <!-- SENSORS -->
+    <xacro:sensor_t265 parent="base_link" name="t265" topics_ns="t265"
+        odom_xyz="0.0 0.0 0.0" odom_rpy="0.0 0.0 0.0" unite_imu_method ="linear_interpolation">
+        <origin xyz="${t265_x_offset} ${t265_y_offset} ${t265_z_offset}" rpy="${t265_x_rotate} ${t265_y_rotate} ${t265_z_rotate}" />
+    </xacro:sensor_t265>
     <xacro:sensor_d435 parent="base_link" name="d435" topics_ns="d435" align_depth="true" enable_pointCloud="true">
         <origin xyz="${d435_x_offset} ${d435_y_offset}  ${d435_z_offset}" rpy="${d435_x_rotate} ${d435_y_rotate}  ${d435_z_rotate}" />

Commit message: add controllers and controller manager

File: src/omnibot_description/urdf/omnibot_description.urdf.xacro (robot description, xacro)
@@ -3,10 +3,52 @@
     <xacro:arg name="use_manipulator" default="false" />
     <xacro:arg name="robot_namespace" default="omnibot_robot" />
-    <xacro:property name="ns" value="$(arg robot_namespace)"/>
+    <xacro:property name="ns" value="$(arg robot_namespace)" />
+    <ros2_control name="GazeboSystem" type="system">
+        <hardware>
+          <plugin>gazebo_ros2_control/GazeboSystem</plugin>
+        </hardware>
+        <joint name="left_front_mecanum_joint">
+            <command_interface name="velocity">
+                <param name="min">-15</param>
+                <param name="max">15</param>
+            </command_interface>
+            <state_interface name="position" />
+            <state_interface name="velocity" />
+            <state_interface name="effort" />
+        </joint>
+        <joint name="right_front_mecanum_joint">
+            <command_interface name="velocity">
+                <param name="min">-15</param>
+                <param name="max">15</param>
+            </command_interface>
+            <state_interface name="position" />
+            <state_interface name="velocity" />
+            <state_interface name="effort" />
+        </joint>
+        <joint name="left_back_mecanum_joint">
+            <command_interface name="velocity">
+                <param name="min">-15</param>
+                <param name="max">15</param>
+            </command_interface>
+            <state_interface name="position" />
+            <state_interface name="velocity" />
+            <state_interface name="effort" />
+        </joint>
+        <joint name="right_back_mecanum_joint">
+            <command_interface name="velocity">
+                <param name="min">-15</param>
+                <param name="max">15</param>
+            </command_interface>
+            <state_interface name="position" />
+            <state_interface name="velocity" />
+            <state_interface name="effort" />
+        </joint>
+    </ros2_control>
     <gazebo>
+        <!-- Joint state publisher -->
         <plugin filename="libgazebo_ros2_control.so" name="gazebo_ros2_control">
-            <robotNamespace>${ns}</robotNamespace>
-            <robot_sim_type>gazebo_ros2_control/GazeboSystem</robot_sim_type>
-             <!-- <parameters>$(find omnibot_gazebo)/config/controller_manager.yaml</parameters> -->
+            <robot_param>robot_description</robot_param>
+            <robot_param_node>robot_state_publisher</robot_param_node>
+            <parameters>$(find omnibot_description)/config/controller_manager.yaml</parameters>
         </plugin>
     </gazebo>

Commit message: add lonk with gazebo and velocity controller

File: src/omnibot_description/urdf/omnibot_description.urdf.xacro (robot description, xacro)
@@ -1,4 +1,7 @@
 <?xml version="1.0"?>
 <robot xmlns:xacro="http://www.ros.org/wiki/xacro" name="omnibot_robot">
+    <xacro:arg name="robot_name" default="omnibot_robot"/>
+    <xacro:include filename="$(find omnibot_description)/urdf/gazebo_sim_ros2_control.urdf.xacro" />
+    <xacro:load_gazebo_sim_ros2_control_plugin robot_name="$(arg robot_name)" use_gazebo="true"/>
     <xacro:include filename="$(find omnibot_platform_description)/urdf/omnibot_platform_description.urdf.xacro" />
 </robot>

File: src/omnibot_platform/omnibot_platform_description/urdf/mecanum_wheel_macro.xacro (robot description, xacro)
@@ -22,4 +22,14 @@
         <limit lower="-3.14" upper="3.14" effort="1000.0" velocity="100.0" />
     </joint>
+    <gazebo>
+      <plugin filename="gz-sim-joint-controller-system" name="gz::sim::systems::JointController">
+                    <joint_name>${name}_mecanum_joint</joint_name>
+                    <topic>${name}_mecanum_joint/velocity</topic>
+                    <initial_velocity>0.0</initial_velocity>
+      </plugin>
+      <plugin  filename="gz-sim-joint-state-publisher-system" name="gz::sim::systems::JointStatePublisher">
+          <joint_name>${name}_mecanum_joint</joint_name>
+      </plugin>
+    </gazebo>
   </xacro:macro>
 </robot>

File: src/omnibot_platform/omnibot_platform_description/urdf/omnibot_platform_description.urdf.xacro (robot description, xacro)
@@ -20,9 +20,17 @@
     <xacro:property name="wheel_offset_y" value="${(wheel_base_width / 2) + 0.035}" />
     <xacro:property name="wheel_offset_z" value="0.015500" />
+    <!-- LIDAR -->
+    <xacro:property name="rplidar_a3_xacro_path" value="rplidar_a3.urdf.xacro" />
+    <xacro:property name="rplidar_a3_x_offset" value="0.168000"/>
+    <xacro:property name="rplidar_a3_y_offset" value="0.0"/>
+    <xacro:property name="rplidar_a3_z_offset" value="${0.148960 - 0.035}"/>
+    <xacro:property name="rplidar_a3_x_rotate" value="0.00"/>
+    <xacro:property name="rplidar_a3_y_rotate" value="0.00"/>
+    <xacro:property name="rplidar_a3_z_rotate" value="1.57"/>
     <!--  INCLUDES -->
     <xacro:include filename="${wheel_macro_path}" />
     <!-- <xacro:include filename="${d435_xacro_path}" /> -->
     <!-- <xacro:include filename="${t265_xacro_path}" /> -->
-    <!-- <xacro:include filename="${rplidar_a3_xacro_path}"/> -->
+    <xacro:include filename="${rplidar_a3_xacro_path}"/>
     <xacro:include filename="$(find omnibot_platform_description)/urdf/inertia_calc.xacro" />
      <!--  PLATFORM DESCRIPTION -->
@@ -77,3 +85,7 @@
             rpy="0.0 0.0 -1.57" />
     </xacro:mecanum_wheel>
+    <xacro:rplidar_a3 suffix="front">
+        <origin xyz="${rplidar_a3_x_offset} ${rplidar_a3_y_offset} ${rplidar_a3_z_offset}" rpy="${rplidar_a3_x_rotate} ${rplidar_a3_y_rotate} ${rplidar_a3_z_rotate}"/>
+        <parent link="base_link"/>
+    </xacro:rplidar_a3>
 </robot>
