Commit message: omnibot_controllers config move to omnibot_platform_control

File: src/omnibot_description/urdf/omnibot_description.urdf.xacro (robot description, xacro)
@@ -2,6 +2,4 @@
 <robot xmlns:xacro="http://www.ros.org/wiki/xacro" name="omnibot_robot">
     <xacro:arg name="robot_name" default="omnibot_robot"/>
-    <xacro:include filename="$(find omnibot_description)/urdf/gazebo_sim_ros2_control.urdf.xacro" />
-    <xacro:load_gazebo_sim_ros2_control_plugin robot_name="$(arg robot_name)" use_gazebo="true"/>
     <xacro:include filename="$(find omnibot_platform_description)/urdf/omnibot_platform_description.urdf.xacro" />
 </robot>

File: src/omnibot_platform/omnibot_platform_description/urdf/omnibot_platform_description.urdf.xacro (robot description, xacro)
@@ -1,7 +1,115 @@
 <?xml version="1.0"?>
 <robot xmlns:xacro="http://www.ros.org/wiki/xacro" name="omnibot_platfrom">
-    <arg name="robot_ns" default="omnibot_robot"/>
+    <arg name="robot_ns" default="omnibot_robot" />
+    <gazebo>
+        <plugin filename="gz_ros2_control-system" name="gz_ros2_control::GazeboSimROS2ControlPlugin">
+            <parameters>$(find omnibot_platform_control)/config/omnibot_platform_ros2_controllers.yaml</parameters>
+        </plugin>
+    </gazebo>
+    <ros2_control name="OmnibotPlatformSystem" type="system">
+        <hardware>
+            <plugin>gz_ros2_control/GazeboSimSystem</plugin>
+        </hardware>
+        <joint name="left_front_mecanum_joint">
+            <command_interface name="velocity">
+                <param name="min">-50.0</param>
+                <param name="max">50.0</param>
+            </command_interface>
+            <state_interface name="position" />
+            <state_interface name="velocity" />
+        </joint>
+        <joint name="right_front_mecanum_joint">
+            <command_interface name="velocity">
+                <param name="min">-50.0</param>
+                <param name="max">50.0</param>
+            </command_interface>
+            <state_interface name="position" />
+            <state_interface name="velocity" />
+        </joint>
+        <joint name="left_back_mecanum_joint">
+            <command_interface name="velocity">
+                <param name="min">-50.0</param>
+                <param name="max">50.0</param>
+            </command_interface>
+            <state_interface name="position" />
+            <state_interface name="velocity" />
+        </joint>
+        <joint name="right_back_mecanum_joint">
+            <command_interface name="velocity">
+                <param name="min">-50.0</param>
+                <param name="max">50.0</param>
+            </command_interface>
+            <state_interface name="position" />
+            <state_interface name="velocity" />
+        </joint>
+    </ros2_control>
+    <gazebo>
+        <plugin filename="gz-sim-joint-state-publisher-system"
+            name="gz::sim::systems::JointStatePublisher">
+            <joint_name>left_front_mecanum_joint</joint_name>
+            <joint_name>left_front_roller_1_7_joint</joint_name>
+            <joint_name>left_front_roller_1_6_joint</joint_name>
+            <joint_name>left_front_roller_1_5_joint</joint_name>
+            <joint_name>left_front_roller_1_4_joint</joint_name>
+            <joint_name>left_front_roller_1_3_joint</joint_name>
+            <joint_name>left_front_roller_1_2_joint</joint_name>
+            <joint_name>left_front_roller_1_1_joint</joint_name>
+            <joint_name>left_front_roller_2_7_joint</joint_name>
+            <joint_name>left_front_roller_2_6_joint</joint_name>
+            <joint_name>left_front_roller_2_5_joint</joint_name>
+            <joint_name>left_front_roller_2_4_joint</joint_name>
+            <joint_name>left_front_roller_2_3_joint</joint_name>
+            <joint_name>left_front_roller_2_2_joint</joint_name>
+            <joint_name>left_front_roller_2_1_joint</joint_name>
+            <joint_name>right_front_mecanum_joint</joint_name>
+            <joint_name>right_front_roller_1_7_joint</joint_name>
+            <joint_name>right_front_roller_1_6_joint</joint_name>
+            <joint_name>right_front_roller_1_5_joint</joint_name>
+            <joint_name>right_front_roller_1_4_joint</joint_name>
+            <joint_name>right_front_roller_1_3_joint</joint_name>
+            <joint_name>right_front_roller_1_2_joint</joint_name>
+            <joint_name>right_front_roller_1_1_joint</joint_name>
+            <joint_name>right_front_roller_2_7_joint</joint_name>
+            <joint_name>right_front_roller_2_6_joint</joint_name>
+            <joint_name>right_front_roller_2_5_joint</joint_name>
+            <joint_name>right_front_roller_2_4_joint</joint_name>
+            <joint_name>right_front_roller_2_3_joint</joint_name>
+            <joint_name>right_front_roller_2_2_joint</joint_name>
+            <joint_name>right_front_roller_2_1_joint</joint_name>
+            <joint_name>left_back_mecanum_joint</joint_name>
+            <joint_name>left_back_roller_1_7_joint</joint_name>
+            <joint_name>left_back_roller_1_6_joint</joint_name>
+            <joint_name>left_back_roller_1_5_joint</joint_name>
+            <joint_name>left_back_roller_1_4_joint</joint_name>
+            <joint_name>left_back_roller_1_3_joint</joint_name>
+            <joint_name>left_back_roller_1_2_joint</joint_name>
+            <joint_name>left_back_roller_1_1_joint</joint_name>
+            <joint_name>left_back_roller_2_7_joint</joint_name>
+            <joint_name>left_back_roller_2_6_joint</joint_name>
+            <joint_name>left_back_roller_2_5_joint</joint_name>
+            <joint_name>left_back_roller_2_4_joint</joint_name>
+            <joint_name>left_back_roller_2_3_joint</joint_name>
+            <joint_name>left_back_roller_2_2_joint</joint_name>
+            <joint_name>left_back_roller_2_1_joint</joint_name>
+            <joint_name>right_back_mecanum_joint</joint_name>
+            <joint_name>right_back_roller_1_7_joint</joint_name>
+            <joint_name>right_back_roller_1_6_joint</joint_name>
+            <joint_name>right_back_roller_1_5_joint</joint_name>
+            <joint_name>right_back_roller_1_4_joint</joint_name>
+            <joint_name>right_back_roller_1_3_joint</joint_name>
+            <joint_name>right_back_roller_1_2_joint</joint_name>
+            <joint_name>right_back_roller_1_1_joint</joint_name>
+            <joint_name>right_back_roller_2_7_joint</joint_name>
+            <joint_name>right_back_roller_2_6_joint</joint_name>
+            <joint_name>right_back_roller_2_5_joint</joint_name>
+            <joint_name>right_back_roller_2_4_joint</joint_name>
+            <joint_name>right_back_roller_2_3_joint</joint_name>
+            <joint_name>right_back_roller_2_2_joint</joint_name>
+            <joint_name>right_back_roller_2_1_joint</joint_name>
+        </plugin>
+    </gazebo>
     <!-- BASE_LINK -->
-    <xacro:property name="base_link_mesh_path" value="file://$(find omnibot_platform_description)/meshes/base_link.dae" />
+    <xacro:property name="base_link_mesh_path"
+        value="file://$(find omnibot_platform_description)/meshes/base_link.dae" />
     <xacro:property name="base_link_offset_x" value="0.0" />
     <xacro:property name="base_link_offset_y" value="0.0" />
@@ -22,18 +130,18 @@
     <!-- LIDAR -->
     <xacro:property name="rplidar_a3_xacro_path" value="rplidar_a3.urdf.xacro" />
-    <xacro:property name="rplidar_a3_x_offset" value="0.168000"/>
-    <xacro:property name="rplidar_a3_y_offset" value="0.0"/>
-    <xacro:property name="rplidar_a3_z_offset" value="${0.148960 - 0.035}"/>
-    <xacro:property name="rplidar_a3_x_rotate" value="0.00"/>
-    <xacro:property name="rplidar_a3_y_rotate" value="0.00"/>
-    <xacro:property name="rplidar_a3_z_rotate" value="1.57"/>
+    <xacro:property name="rplidar_a3_x_offset" value="0.168000" />
+    <xacro:property name="rplidar_a3_y_offset" value="0.0" />
+    <xacro:property name="rplidar_a3_z_offset" value="${0.148960 - 0.035}" />
+    <xacro:property name="rplidar_a3_x_rotate" value="0.00" />
+    <xacro:property name="rplidar_a3_y_rotate" value="0.00" />
+    <xacro:property name="rplidar_a3_z_rotate" value="1.57" />
     <!--  INCLUDES -->
     <xacro:include filename="${wheel_macro_path}" />
     <!-- <xacro:include filename="${d435_xacro_path}" /> -->
     <!-- <xacro:include filename="${t265_xacro_path}" /> -->
-    <xacro:include filename="${rplidar_a3_xacro_path}"/>
+    <xacro:include filename="${rplidar_a3_xacro_path}" />
     <xacro:include filename="$(find omnibot_platform_description)/urdf/inertia_calc.xacro" />
-     <!--  PLATFORM DESCRIPTION -->
-    <link name="base_footprint"/>
+    <!--  PLATFORM DESCRIPTION -->
+    <link name="base_footprint" />
     <link name="base_link">
         <inertial>
@@ -86,6 +194,7 @@
     </xacro:mecanum_wheel>
     <xacro:rplidar_a3 suffix="front">
-        <origin xyz="${rplidar_a3_x_offset} ${rplidar_a3_y_offset} ${rplidar_a3_z_offset}" rpy="${rplidar_a3_x_rotate} ${rplidar_a3_y_rotate} ${rplidar_a3_z_rotate}"/>
-        <parent link="base_link"/>
+        <origin xyz="${rplidar_a3_x_offset} ${rplidar_a3_y_offset} ${rplidar_a3_z_offset}"
+            rpy="${rplidar_a3_x_rotate} ${rplidar_a3_y_rotate} ${rplidar_a3_z_rotate}" />
+        <parent link="base_link" />
     </xacro:rplidar_a3>
 </robot>

File: src/omnibot_platform/omnibot_platform_description/urdf/rplidar_a3.urdf.xacro (robot description, xacro)
@@ -44,8 +44,4 @@
                     <mesh filename="file://$(find omnibot_platform_description)/meshes/rplidarA3.dae" scale="0.001 0.001 0.001"/>
                 </geometry>
-                <material name="">
-                    <color rgba="1.0 1.0 0.0 1.0" />
-                    <texture filename="" />
-                </material>
             </visual>
             <collision>
