Commit message: fix manipulator moveit package

File: src/omnibot_manipulator/urdf/angle_arm.urdf (robot description, URDF)
Before this commit: robot angle_robot, 9 links, 8 joints
Links:
- added link tip_link
Joints:
- added joint tip_joint: type fixed, parent ang_link5, child tip_link, origin xyz=0.0 0.0 -0.1 rpy=0.0 0.0 0.0, axis 0.0 0.0 0.0, limit lower=0.0 upper=0.0 effort=0.0 velocity=0.0
- joint ang_gripper: origin xyz=0 0 -0.0715 rpy=1.57 3.14 0 -> xyz=0.0 0.0 0.0285 rpy=1.57 3.14 0; parent ang_link5 -> tip_link
- joint ang_gripper_sub: origin xyz=0 0 -0.0715 rpy=-1.57 0 0 -> xyz=0.0 0.0 0.0285 rpy=-1.57 0 0; parent ang_link5 -> tip_link
- joint ang_joint2: limit effort=5.0 velocity=5.0 -> lower=-1.57 upper=1.57 effort=5.0 velocity=5.0; type continuous -> revolute
- joint ang_joint3: limit effort=5.0 velocity=5.0 -> lower=-1.57 upper=1.57 effort=5.0 velocity=5.0; type continuous -> revolute
- joint ang_joint4: limit effort=5.0 velocity=5.0 -> lower=-1.45 upper=1.45 effort=5.0 velocity=5.0; type continuous -> revolute
- joint ang_joint5: limit effort=5.0 velocity=5.0 -> lower=-1.57 upper=1.57 effort=5.0 velocity=5.0

Commit message: add robot_description and test moveit package

File: src/omnibot_manipulator/urdf/angle_arm.urdf (robot description, URDF)
Before this commit: robot angle_robot, 10 links, 9 joints
Links:
- removed link map
Joints:
- removed joint ang_base

Commit message: remake omnibot moveit pkg, but not working

File: src/omnibot_manipulator/urdf/angle_arm.urdf (robot description, URDF)
Before this commit: robot angle_robot, 9 links, 8 joints
Links:
- link ang_link0: mass 1 -> None

File: src/omnibot_platform/urdf/platform.urdf.xacro (robot description, xacro)
@@ -6,5 +6,6 @@
     <xacro:property name="wheel_x_offset" value="${(base_lenth / 2) + 0.03}" />
     <xacro:property name="wheel_y_offset" value="${(base_width / 2)}" />
-    <xacro:macro name="wheel_caster" params="suffix *origin">
+    <!-- wheel template -->
+    <xacro:macro name="wheel_template" params="suffix *origin">
         <link name="${suffix}_wheel_link">
             <visual name="">
@@ -25,12 +26,23 @@
             </collision>
         </link>
-        <joint name="${suffix}_wheel_joint" type="fixed">
+        <joint name="${suffix}_wheel_joint" type="continuous">
             <xacro:insert_block name="origin" />
             <parent link="base_link" />
             <child link="${suffix}_wheel_link" />
-            <axis xyz="0.0 0.0 0.0" />
+            <axis xyz="1.0 0.0 0.0" />
             <limit effort="0.0" velocity="0.0" />
         </joint>
+        <transmission name="${suffix}_wheel_trans" type="SimpleTransmission">
+            <type>transmission_interface/SimpleTransmission</type>
+            <actuator name="${suffix}_wheel_motor">
+                <hardwareInterface>hardware_interface/VelocityJointInterface</hardwareInterface>
+                <mechanicalReduction>1</mechanicalReduction>
+            </actuator>
+            <joint name="${suffix}_wheel_joint">
+                <hardwareInterface>hardware_interface/VelocityJointInterface</hardwareInterface>
+            </joint>
+        </transmission>
     </xacro:macro>
+    <!-- #######################################################################################################333333333 -->
     <link name="base_link">
         <visual name="">
@@ -51,15 +63,15 @@
         </collision>
     </link>
-    <xacro:wheel_caster suffix="right_forward">
+    <xacro:wheel_template suffix="left_forward">
+        <origin xyz="${-wheel_x_offset} ${wheel_y_offset} 0.0" rpy="0.0 0.0 0.0" />
+    </xacro:wheel_template>
+    <xacro:wheel_template suffix="right_forward">
         <origin xyz="${wheel_x_offset} ${wheel_y_offset} 0.0" rpy="0.0 0.0 0.0" />
-    </xacro:wheel_caster>
-    <xacro:wheel_caster suffix="left_forward">
-        <origin xyz="${-wheel_x_offset} ${wheel_y_offset} 0.0" rpy="0.0 0.0 0.0" />
-    </xacro:wheel_caster>
-    <xacro:wheel_caster suffix="left_backward">
+    </xacro:wheel_template>
+    <xacro:wheel_template suffix="left_backward">
         <origin xyz="${-wheel_x_offset} ${-wheel_y_offset} 0.0" rpy="0.0 0.0 0.0" />
-    </xacro:wheel_caster>
-    <xacro:wheel_caster suffix="right_backward">
+    </xacro:wheel_template>
+    <xacro:wheel_template suffix="right_backward">
         <origin xyz="${wheel_x_offset} ${-wheel_y_offset} 0.0" rpy="0.0 0.0 0.0" />
-    </xacro:wheel_caster>
+    </xacro:wheel_template>
 </robot>

Commit message: add gazebo model

File: src/omnibot_manipulator/urdf/angle_arm.urdf (robot description, URDF)
Before this commit: robot angle_robot, 9 links, 8 joints
Links:
- link ang_link0: mass None -> 1

File: src/omnibot_platform/urdf/platform.urdf.xacro (robot description, xacro)
@@ -6,5 +6,4 @@
     <xacro:property name="wheel_x_offset" value="${(base_lenth / 2)}" />
     <xacro:property name="wheel_y_offset" value="${(base_width / 2)}" />
-    <!-- wheel template -->
     <xacro:macro name="wheel_template" params="suffix *origin">
         <link name="${suffix}_wheel_link">
@@ -12,5 +11,5 @@
                 <origin xyz="0.0 0.0 0.0" rpy="0.0 0.0 0.0" />
                 <geometry>
-                    <mesh filename="package://omnibot_platform/meshes/wheel.STL" scale="0.001 0.001 0.001" />
+                    <mesh filename="package://omnibot_platform/meshes/wheel_low.dae" scale="0.001 0.001 0.001" />
                 </geometry>
                 <material name="">
@@ -22,5 +21,5 @@
                 <origin xyz="0.0 0.0 0.0" rpy="0.0 0.0 0.0" />
                 <geometry>
-                    <mesh filename="package://omnibot_platform/meshes/wheel.STL" scale="0.001 0.001 0.001" />
+                    <mesh filename="package://omnibot_platform/meshes/wheel_low.dae" scale="0.001 0.001 0.001" />
                 </geometry>
             </collision>
@@ -33,5 +32,5 @@
             <limit effort="0.0" velocity="0.0" />
         </joint>
-        <transmission name="${suffix}_wheel_trans" type="SimpleTransmission">
+        <transmission name="${suffix}_wheel_transmission" type="SimpleTransmission">
             <type>transmission_interface/SimpleTransmission</type>
             <actuator name="${suffix}_wheel_motor">
@@ -44,10 +43,9 @@
         </transmission>
     </xacro:macro>
-    <!-- #######################################################################################################333333333 -->
     <link name="base_link">
         <visual name="">
-            <origin xyz="0.0 0.0 0.0" rpy="-1.57 0.0 3.14" />
+            <origin xyz="0.0 0.0 0.0" rpy="0.0 3.14 0.0" />
             <geometry>
-                <mesh filename="package://omnibot_platform/meshes/base.STL" scale="0.001 0.001 0.001"/>
+                <mesh filename="package://omnibot_platform/meshes/hodovaya_low.dae" scale="0.001 0.001 0.001"/>
             </geometry>
             <material name="">
@@ -59,19 +57,19 @@
             <origin xyz="0.0 0.0 0.0" rpy="0.0 0.0 0.0" />
             <geometry>
-                <mesh filename="package://omnibot_platform/meshes/base.STL" scale="0.001 0.001 0.001"/>
+                <mesh filename="package://omnibot_platform/meshes/hodovaya_low.dae" scale="0.001 0.001 0.001"/>
             </geometry>
         </collision>
     </link>
     <xacro:wheel_template suffix="left_forward">
-        <origin xyz="${-wheel_x_offset} ${wheel_y_offset} 0.013285" rpy="0.0 1.57 0.0" />
+        <origin xyz="${-wheel_x_offset} ${wheel_y_offset} 0.013285" rpy="0.0 0.0 1.57" />
     </xacro:wheel_template>
     <xacro:wheel_template suffix="right_forward">
-        <origin xyz="${wheel_x_offset} ${wheel_y_offset} 0.013285" rpy="0.0 -1.57 0.0" />
+        <origin xyz="${wheel_x_offset} ${wheel_y_offset} 0.013285" rpy="0.0 0.0 1.57" />
     </xacro:wheel_template>
     <xacro:wheel_template suffix="left_backward">
-        <origin xyz="${-wheel_x_offset} ${-wheel_y_offset} 0.013285" rpy="0.0 1.57 0.0" />
+        <origin xyz="${-wheel_x_offset} ${-wheel_y_offset} 0.013285" rpy="0.0 0.0  1.57" />
     </xacro:wheel_template>
     <xacro:wheel_template suffix="right_backward">
-        <origin xyz="${wheel_x_offset} ${-wheel_y_offset} 0.013285" rpy="0.0 -1.57 0.0" />
+        <origin xyz="${wheel_x_offset} ${-wheel_y_offset} 0.013285" rpy="0.0 0.0  1.57" />
     </xacro:wheel_template>
 </robot>
