Commit message: add teleop pkg

File: src/omnibot_platform/omnibot_platform_description/urdf/mecanum_wheel_macro.xacro (robot description, xacro)
@@ -12,5 +12,5 @@
         </actuator>
         <joint name="${name}_mecanum_joint">
-            <hardwareInterface>hardware_interface/VelocityJointInterface</hardwareInterface>
+            <hardwareInterface>${interface}</hardwareInterface>
         </joint>
     </transmission>
@@ -20,5 +20,5 @@
         <child link="${name}_mecanum_wheel_link" />
         <axis xyz="1 0 0" />
-        <limit lower="-3.14" upper="3.14" effort="1000.0" velocity="50.0" />
+        <limit lower="-3.14" upper="3.14" effort="1000.0" velocity="100.0" />
     </joint>
   </xacro:macro>

File: src/omnibot_platform/omnibot_platform_description/urdf/omnibot_platform.urdf.xacro (robot description, xacro)
@@ -94,20 +94,20 @@
     </xacro:omniwheel_macro> -->
     <xacro:mecanum_wheel name="left_front" side="1"
-        interface="hardware_interface/EffortJointInterface">
+        interface="hardware_interface/VelocityJointInterface">
         <origin xyz="${omniwheel_offset_x} ${omniwheel_offset_y} ${omniwheel_offset_z}"
             rpy="0.0 0.0 1.57" />
     </xacro:mecanum_wheel>
     <xacro:mecanum_wheel name="right_front" side="-1"
-        interface="hardware_interface/EffortJointInterface">
+        interface="hardware_interface/VelocityJointInterface">
         <origin xyz="${omniwheel_offset_x} ${-omniwheel_offset_y} ${omniwheel_offset_z}"
             rpy="0.0 0.0 1.57" />
     </xacro:mecanum_wheel>
     <xacro:mecanum_wheel name="left_back" side="-1"
-        interface="hardware_interface/EffortJointInterface">
+        interface="hardware_interface/VelocityJointInterface">
         <origin xyz="${-omniwheel_offset_x} ${omniwheel_offset_y} ${omniwheel_offset_z}"
             rpy="0.0 0.0 -1.57" />
     </xacro:mecanum_wheel>
     <xacro:mecanum_wheel name="right_back" side="1"
-        interface="hardware_interface/EffortJointInterface">
+        interface="hardware_interface/VelocityJointInterface">
         <origin xyz="${-omniwheel_offset_x} ${-omniwheel_offset_y} ${omniwheel_offset_z}"
             rpy="0.0 0.0 -1.57" />

File: src/omnibot_platform/omnibot_platform_description/urdf/rollers.xacro (robot description, xacro)
@@ -43,4 +43,23 @@
                   izz="0.00076000" />
         </inertial>
+        <surface>
+          <friction>
+            <ode>
+              <mu1>1.2</mu1>
+              <mu2>1.2</mu2>
+              <kp>1e15</kp>
+              <kd>1e13</kd>
+            </ode>
+          </friction>
+          <bounce>
+            <restitution_coefficient>0.01</restitution_coefficient>
+            <threshold>0</threshold>
+          </bounce>
+          <contact>
+            <ode>
+              <max_vel>10</max_vel>
+            </ode>
+          </contact>
+        </surface>
       </link>
       <joint name="${joint_name}_joint" type="continuous">
@@ -51,5 +70,5 @@
         <dynamics damping="0.001" friction="0.0001" />
       </joint>
-      <transmission name="$${joint_name}_trans">
+      <transmission name="${joint_name}_trans">
         <type>transmission_interface/SimpleTransmission</type>
         <joint name="${joint_name}_joint">
@@ -62,10 +81,8 @@
       </transmission>
       <gazebo reference="${joint_name}_link">
-        <mu1 value="0.8"/>
-        <mu2 value="0.8"/>
-        <kp value="10000000.0" />
-        <kd value="1.0" />
-        <fdir1 value="0 1 0"/>
-      </gazebo>
+        <selfCollide>false</selfCollide>
+          <mu1 value="1.2" />
+          <mu2 value="1.2" />
+        </gazebo>
       <xacro:roller_loop name="${name}" side="${side}" num="${num}" loop="${loop - 1}"  wheel_side2="${wheel_side2}"/>
     </xacro:if>

File: src/omnibot_platform/omnibot_platform_description/urdf/wheel.xacro (robot description, xacro)
@@ -6,5 +6,5 @@
         <origin xyz="0 0 0" rpy="0 0 ${1.57 * side}" />
         <geometry>
-          <mesh filename="package://omnibot_platform_description/meshes/meccanum_wheel3.dae" scale="${side / 1000} 0.001 0.001" />
+          <mesh filename="package://omnibot_platform_description/meshes/wheel_base.dae" scale="${side / 1000} 0.001 0.001" />
         </geometry>
       </visual>
@@ -12,13 +12,37 @@
         <origin xyz="0 0 0" rpy="0 0 ${1.57 * side}" />
         <geometry>
-          <mesh filename="package://omnibot_platform_description/meshes/meccanum_wheel3.dae" scale="${side / 1000} 0.001 0.001" />
+          <mesh filename="package://omnibot_platform_description/meshes/wheel_base.dae" scale="${side / 1000} 0.001 0.001" />
         </geometry>
       </collision>
       <inertial>
-        <origin xyz="0 0 0" rpy="0 0 ${1.57 * side}" />
-        <mass value="2.0" />
-        <inertia ixx="0.042025" ixy="0.0" ixz="0.0"
-                iyy="0.024279" iyz="0.0"
-                izz="0.024279" />
+        <origin xyz="0 0 0" rpy="0 0 0" />
+        <mass value="0.25"/>
+        <inertia ixx="0.00031" ixy="0" ixz="0" iyy="0.0005" iyz="0" izz="0.00031"/>
+      </inertial>
+    </link>
+    <joint name="${name}_adapter_connector_joint" type="fixed">
+      <parent link="${name}_mecanum_wheel_link"/>
+      <child link="${name}_mecanum_adapter_link"/>
+      <origin xyz="0 0 0" rpy="0 0 ${1.57 * side}" />
+    </joint>
+    <link name="${name}_mecanum_adapter_link">
+      <visual>
+        <origin xyz="0 0.035 0" rpy="0 0 ${1.57 * side}" />
+        <geometry>
+          <mesh filename="package://omnibot_platform_description/meshes/adapter.dae" scale="${side / 1000} 0.001 0.001" />
+        </geometry>
+      </visual>
+      <collision>
+        <origin xyz="0 0.035 0" rpy="0 0 ${1.57 * side}" />
+        <geometry>
+          <mesh filename="package://omnibot_platform_description/meshes/adapter.dae" scale="${side / 1000} 0.001 0.001" />
+        </geometry>
+      </collision>
+      <inertial>
+        <origin xyz="0 0 0" rpy="0 0 0" />
+        <mass value="0.005" />
+        <inertia ixx="0.00001" ixy="0.0" ixz="0.0"
+                iyy="0.00001" iyz="0.0"
+                izz="0.00001" />
       </inertial>
     </link>

Commit message: some fixes in gazebo pkg

File: src/omnibot_platform/omnibot_platform_description/urdf/mecanum_wheel_macro.xacro (robot description, xacro)
@@ -15,5 +15,5 @@
         </joint>
     </transmission>
-    <joint name="${name}_mecanum_joint" type="revolute">
+    <joint name="${name}_mecanum_joint" type="continuous">
         <xacro:insert_block name="origin" />
         <parent link="base_link" />

File: src/omnibot_platform/omnibot_platform_description/urdf/rollers.xacro (robot description, xacro)
@@ -46,6 +46,6 @@
           <friction>
             <ode>
-              <mu1>1.2</mu1>
-              <mu2>1.2</mu2>
+              <mu1>10.2</mu1>
+              <mu2>10.2</mu2>
               <kp>1e15</kp>
               <kd>1e13</kd>
@@ -58,5 +58,5 @@
           <contact>
             <ode>
-              <max_vel>10</max_vel>
+              <max_vel>100</max_vel>
             </ode>
           </contact>
