Commit message: fix odom bugs, add sensor odom manager package

File: src/omnibot_platform/omnibot_platform_description/urdf/d435.urdf.xacro (robot description, xacro)
@@ -3,70 +3,82 @@
 The MIT License
 Copyright (c) 2019 Giovanni di Dio Bruno https://gbr1.github.io
-Permission is hereby granted, free of charge, to any person obtaining a copy
-of this software and associated documentation files (the "Software"), to deal
-in the Software without restriction, including without limitation the rights
+Permission is
+hereby granted, free of charge, to any person obtaining a copy
+of this software and associated
+documentation files (the "Software"), to deal
+in the Software without restriction, including without
+limitation the rights
 to use, copy, modify, merge, publish, distribute, sublicense, and/or sell
 copies of the Software, and to permit persons to whom the Software is
-furnished to do so, subject to the following conditions:
-The above copyright notice and this permission notice shall be included in
+furnished to do so, subject to
+the following conditions:
+The above copyright notice and this permission notice shall be included
+in
 all copies or substantial portions of the Software.
-THE SOFTWARE IS PROVIDED "AS IS", WITHOUT WARRANTY OF ANY KIND, EXPRESS OR
-IMPLIED, INCLUDING BUT NOT LIMITED TO THE WARRANTIES OF MERCHANTABILITY,
+THE SOFTWARE IS PROVIDED "AS IS", WITHOUT
+WARRANTY OF ANY KIND, EXPRESS OR
+IMPLIED, INCLUDING BUT NOT LIMITED TO THE WARRANTIES OF
+MERCHANTABILITY,
 FITNESS FOR A PARTICULAR PURPOSE AND NONINFRINGEMENT. IN NO EVENT SHALL THE
-AUTHORS OR COPYRIGHT HOLDERS BE LIABLE FOR ANY CLAIM, DAMAGES OR OTHER
-LIABILITY, WHETHER IN AN ACTION OF CONTRACT, TORT OR OTHERWISE, ARISING FROM,
-OUT OF OR IN CONNECTION WITH THE SOFTWARE OR THE USE OR OTHER DEALINGS IN
+AUTHORS
+OR COPYRIGHT HOLDERS BE LIABLE FOR ANY CLAIM, DAMAGES OR OTHER
+LIABILITY, WHETHER IN AN ACTION OF
+CONTRACT, TORT OR OTHERWISE, ARISING FROM,
+OUT OF OR IN CONNECTION WITH THE SOFTWARE OR THE USE OR
+OTHER DEALINGS IN
 THE SOFTWARE.
 -->
-<robot name="d435" xmlns:xacro="http://ros.org/wiki/xacro">
-    <xacro:macro name="d435" params="offset_x offset_y offset_z mesh_path">
+<robot name="d400" xmlns:xacro="http://ros.org/wiki/xacro">
+    <xacro:macro name="d400" params="mesh_path parent_link *origin">
         <xacro:property name="M_PI" value="3.1415926535897931" />
         <xacro:property name="M_PI_2" value="1.570796327" />
-        <xacro:property name="d435_cam_depth_to_left_ir_offset" value="0.0"/>
-        <xacro:property name="d435_cam_depth_to_right_ir_offset" value="-0.050"/>
-        <xacro:property name="d435_cam_depth_to_color_offset" value="0.015"/>
-        <xacro:property name="d435_cam_width" value="0.090"/>
-        <xacro:property name="d435_cam_height" value="0.025"/>
-        <xacro:property name="d435_cam_depth" value="0.02505"/>
-        <xacro:property name="d435_cam_mount_from_center_offset" value="0.0149"/>
-        <xacro:property name="d435_cam_depth_px" value="${d435_cam_mount_from_center_offset}"/>
-        <xacro:property name="d435_cam_depth_py" value="0.0175"/>
-        <xacro:property name="d435_cam_depth_pz" value="${d435_cam_height/2}"/>
+        <xacro:property name="d400_cam_depth_to_left_ir_offset" value="0.0" />
+        <xacro:property name="d400_cam_depth_to_right_ir_offset" value="-0.050" />
+        <xacro:property name="d400_cam_depth_to_color_offset" value="0.015" />
+        <xacro:property name="d400_cam_width" value="0.090" />
+        <xacro:property name="d400_cam_height" value="0.025" />
+        <xacro:property name="d400_cam_depth" value="0.02505" />
+        <xacro:property name="d400_cam_mount_from_center_offset" value="0.0149" />
+        <xacro:property name="d400_cam_depth_px" value="${d400_cam_mount_from_center_offset}" />
+        <xacro:property name="d400_cam_depth_py" value="0.0175" />
+        <xacro:property name="d400_cam_depth_pz" value="${d400_cam_height/2}" />
         <joint name="d400_joint" type="fixed">
-            <parent link="base_link"/>
+            <parent link="${parent_link}" />
             <child link="d400_bottom_screw_frame" />
-            <origin rpy="0.0 0.0 0" xyz="${offset_x} ${offset_y} ${offset_z}"/>
-        </joint>
-        <link name="d400_bottom_screw_frame"/>
+            <xacro:insert_block name="origin" />
+        </joint>
+        <link name="d400_bottom_screw_frame" />
         <gazebo reference="d400_bottom_screw_frame">
             <turnGravityOff>false</turnGravityOff>
         </gazebo>
         <joint name="d400_link_joint" type="fixed">
-            <origin xyz="0 ${d435_cam_depth_py} ${d435_cam_depth_pz}" rpy="0 0 0"/>
-            <parent link="d400_bottom_screw_frame"/>
+            <origin xyz="0 ${d400_cam_depth_py} ${d400_cam_depth_pz}" rpy="0 0 0" />
+            <parent link="d400_bottom_screw_frame" />
             <child link="d400_link" />
         </joint>
         <link name="d400_link">
             <visual>
-                <origin xyz="${d435_cam_mount_from_center_offset} ${-d435_cam_depth_py} 0" rpy="${M_PI_2} 0 ${M_PI_2}"/>
+                <origin xyz="${d400_cam_mount_from_center_offset} ${-d400_cam_depth_py} 0"
+                    rpy="${M_PI_2} 0 ${M_PI_2}" />
                 <geometry>
                     <mesh filename="${mesh_path}" scale="0.001 0.001 0.001" />
                 </geometry>
-            <material name="">
-                    <color rgba="0.3 0.3 0.3 1.0"/>
-                    <texture filename=""/>
-            </material>
-        </visual>
-        <collision>
-            <origin xyz="0 ${-d435_cam_depth_py} 0" rpy="0 0 0"/>
-            <geometry>
-                <box size="${d435_cam_depth} ${d435_cam_width} ${d435_cam_height}"/>
-            </geometry>
-        </collision>
-        <inertial>
-            <mass value="0.180" />
-            <origin xyz="0 0 0" />
-            <inertia ixx="0.003881243" ixy="0.0" ixz="0.0" iyy="0.000498940" iyz="0.0" izz="0.003879257" />
-        </inertial>
+                <material name="">
+                    <color rgba="0.3 0.3 0.3 1.0" />
+                    <texture filename="" />
+                </material>
+            </visual>
+            <collision>
+                <origin xyz="0 ${-d400_cam_depth_py} 0" rpy="0 0 0" />
+                <geometry>
+                    <box size="${d400_cam_depth} ${d400_cam_width} ${d400_cam_height}" />
+                </geometry>
+            </collision>
+            <inertial>
+                <mass value="0.180" />
+                <origin xyz="0 0 0" />
+                <inertia ixx="0.003881243" ixy="0.0" ixz="0.0" iyy="0.000498940" iyz="0.0"
+                    izz="0.003879257" />
+            </inertial>
         </link>
         <gazebo reference="d400_link">
@@ -76,9 +88,9 @@
         <!-- d400 depth joints and links -->
         <joint name="d400_depth_joint" type="fixed">
-            <origin xyz="0 0 0" rpy="0 0 0"/>
-            <parent link="d400_link"/>
+            <origin xyz="0 0 0" rpy="0 0 0" />
+            <parent link="d400_link" />
             <child link="d400_depth_frame" />
         </joint>
-        <link name="d400_depth_frame"/>
+        <link name="d400_depth_frame" />
         <gazebo reference="d400_depth_frame">
             <turnGravityOff>false</turnGravityOff>
@@ -89,5 +101,5 @@
             <child link="d400_depth_optical_frame" />
         </joint>
-        <link name="d400_depth_optical_frame"/>
+        <link name="d400_depth_optical_frame" />
         <gazebo reference="d400_depth_optical_frame">
             <turnGravityOff>false</turnGravityOff>
@@ -95,9 +107,9 @@
         <!-- d400 left IR joints and links -->
         <joint name="d400_left_ir_joint" type="fixed">
-            <origin xyz="0 ${d435_cam_depth_to_left_ir_offset} 0" rpy="0 0 0" />
+            <origin xyz="0 ${d400_cam_depth_to_left_ir_offset} 0" rpy="0 0 0" />
             <parent link="d400_depth_frame" />
             <child link="d400_left_ir_frame" />
         </joint>
-        <link name="d400_left_ir_frame"/>
+        <link name="d400_left_ir_frame" />
         <gazebo reference="d400_left_ir_frame">
             <turnGravityOff>false</turnGravityOff>
@@ -108,5 +120,5 @@
             <child link="d400_left_ir_optical_frame" />
         </joint>
-        <link name="d400_left_ir_optical_frame"/>
+        <link name="d400_left_ir_optical_frame" />
         <gazebo reference="d400_left_ir_optical_frame">
             <turnGravityOff>false</turnGravityOff>
@@ -114,9 +126,9 @@
         <!-- d400 right IR joints and links -->
         <joint name="d400_right_ir_joint" type="fixed">
-            <origin xyz="0 ${d435_cam_depth_to_right_ir_offset} 0" rpy="0 0 0" />
+            <origin xyz="0 ${d400_cam_depth_to_right_ir_offset} 0" rpy="0 0 0" />
             <parent link="d400_depth_frame" />
             <child link="d400_right_ir_frame" />
         </joint>
-        <link name="d400_right_ir_frame"/>
+        <link name="d400_right_ir_frame" />
         <gazebo reference="d400_right_ir_frame">
             <turnGravityOff>false</turnGravityOff>
@@ -127,5 +139,5 @@
             <child link="d400_right_ir_optical_frame" />
         </joint>
-        <link name="d400_right_ir_optical_frame"/>
+        <link name="d400_right_ir_optical_frame" />
         <gazebo reference="d400_right_ir_optical_frame">
             <turnGravityOff>false</turnGravityOff>
@@ -133,9 +145,9 @@
         <!-- d400 color joints and links -->
         <joint name="d400_color_joint" type="fixed">
-            <origin xyz="0 ${d435_cam_depth_to_color_offset} 0" rpy="0 0 0" />
+            <origin xyz="0 ${d400_cam_depth_to_color_offset} 0" rpy="0 0 0" />
             <parent link="d400_depth_frame" />
             <child link="d400_color_frame" />
         </joint>
-        <link name="d400_color_frame"/>
+        <link name="d400_color_frame" />
         <gazebo reference="d400_color_frame">
             <turnGravityOff>false</turnGravityOff>
@@ -146,9 +158,9 @@
             <child link="d400_color_optical_frame" />
         </joint>
-        <link name="d400_color_optical_frame"/>
+        <link name="d400_color_optical_frame" />
         <gazebo reference="d400_color_optical_frame">
             <turnGravityOff>false</turnGravityOff>
         </gazebo>
-        <link name="d400_depth_frame_gazebo"/>
+        <link name="d400_depth_frame_gazebo" />
         <joint name="gazebo_joint" type="fixed">
             <origin xyz="0 0 0" rpy="${-M_PI_2} 0 ${-M_PI_2}" />
@@ -161,7 +173,7 @@
     </xacro:macro>
     <gazebo reference="d400_link">
-        <sensor name="d435" type="depth">
+        <sensor name="d400" type="depth">
             <update_rate>30</update_rate>
-            <d400>
+            <camera>
                 <horizontal_fov>1.59174</horizontal_fov>
                 <image>
@@ -174,15 +186,15 @@
                     <far>6</far>
                 </clip>
-            </d400>
+            </camera>
             <plugin name="camera_plugin" filename="libgazebo_ros_openni_kinect.so">
                 <visualize>true</visualize>
                 <baseline>0.05</baseline>
                 <alwaysOn>true</alwaysOn>
-                <updateRate>0.0</updateRate>
-                <cameraName>d435</cameraName>
+                <updateRate>30.0</updateRate>
+                <cameraName>d400</cameraName>
                 <imageTopicName>/d400/color/image_raw</imageTopicName>
                 <cameraInfoTopicName>/d400/color/camera_info</cameraInfoTopicName>
                 <depthImageTopicName>/d400/aligned_depth_to_color/image_raw</depthImageTopicName>
-                <depthImageInfoTopicName>/d400/depth/camera_info</depthImageInfoTopicName>
+                <depthImageInfoTopicName>/d400/depth/d400_info</depthImageInfoTopicName>
                 <pointCloudTopicName>/d400/depth/color/points</pointCloudTopicName>
                 <frameName>d400_depth_frame_gazebo</frameName>

File: src/omnibot_platform/omnibot_platform_description/urdf/mecanum_wheel_macro.xacro (robot description, xacro)
@@ -3,5 +3,5 @@
   <xacro:include filename="$(find omnibot_platform_description)/urdf/wheel.xacro" />
   <xacro:include filename="$(find omnibot_platform_description)/urdf/rollers.xacro"  />
-  <xacro:macro name="mecanum_wheel" params="name side interface *origin">
+  <xacro:macro name="mecanum_wheel" params="name side interface *origin parent">
     <xacro:wheel_link name="${name}" side="${side}" />
     <xacro:rollers_link name="${name}" side="${side}" />
@@ -17,5 +17,5 @@
     <joint name="${name}_mecanum_joint" type="continuous">
         <xacro:insert_block name="origin" />
-        <parent link="base_link" />
+        <parent link="${parent}" />
         <child link="${name}_mecanum_wheel_link" />
         <axis xyz="1 0 0" />

File: src/omnibot_platform/omnibot_platform_description/urdf/omnibot_platform.urdf.xacro (robot description, xacro)
@@ -6,4 +6,13 @@
         </plugin>
     </gazebo>
+    <!-- <gazebo>
+        <plugin name="object_controller" filename="libgazebo_ros_planar_move.so">
+    <commandTopic>cmd_vel</commandTopic>
+            <odometryTopic>odom</odometryTopic>
+    <odometryFrame>odom</odometryFrame>
+            <odometryRate>20.0</odometryRate>
+    <robotBaseFrame>base_link</robotBaseFrame>
+        </plugin>
+    </gazebo> -->
     <!-- BASELINK  -->
     <xacro:property name="wheel_base_width" value="0.306100" />
@@ -24,30 +33,44 @@
     <xacro:property name="omniwheel_offset_y" value="${(wheel_base_width / 2) + 0.035}" />
     <xacro:property name="omniwheel_offset_z" value="0.015500" />
-    <!--
-    <xacro:property name="omniwheel_macro_path"
-            value="$(find
-    omnibot_platform_description)/urdf/omniwheel.urdf.xacro" /> -->
     <xacro:property name="omniwheel_macro_path"
         value="$(find omnibot_platform_description)/urdf/mecanum_wheel_macro.xacro" />
     <!-- REALSENSE -->
-    <xacro:property name="rs435_macro_path"
+<!--
+    <xacro:property name="t265_xacro_path"
+        value="$(find omnibot_platform_description)/urdf/t265.xacro" />
+    <xacro:property name="t265_mesh_path"
+        value="package://omnibot_platform_description/meshes/t265.stl" /> -->
+    <xacro:property name="t265_xacro_path"
+        value="$(find realsense_gazebo_description)/urdf/_t265.urdf.xacro" />
+    <xacro:property name="t265_x_offset" value="0.226500" />
+    <xacro:property name="t265_y_offset" value="0.0" />
+    <xacro:property name="t265_z_offset" value="0.094250" />
+    <!-- <xacro:property name="d435_xacro_path"
         value="$(find omnibot_platform_description)/urdf/d435.urdf.xacro" />
-    <xacro:property name="rs265_macro_path"
-        value="$(find omnibot_platform_description)/urdf/tracker.xacro" />
-    <xacro:property name="rs_d435_mesh_path"
-        value="package://omnibot_platform_description/meshes/d435.STL" />
-    <xacro:property name="rs_t265_mesh_path"
-        value="package://omnibot_platform_description/meshes/t265.STL" />
+    <xacro:property name="d435_mesh_path"
+        value="package://omnibot_platform_description/meshes/d435.stl" /> -->
+    <xacro:property name="d435_xacro_path"
+        value="$(find realsense_gazebo_description)/urdf/_d435.urdf.xacro" />
+    <xacro:property name="d435_x_offset" value="${0.196 + 0.0105 + 0.005}" />
+    <xacro:property name="d435_y_offset" value="0.0" />
+    <xacro:property name="d435_z_offset" value="0.114" />
+    <!-- <xacro:property name="d435_x_offset" value="-0.01950" />
+    <xacro:property name="d435_y_offset" value="0.0" />
+    <xacro:property name="d435_z_offset" value="0.019" /> -->
     <!--  INCLUDES -->
     <xacro:include filename="${omniwheel_macro_path}" />
-    <xacro:include filename="${rs435_macro_path}" />
-    <xacro:include filename="${rs265_macro_path}" />
+    <xacro:include filename="${d435_xacro_path}" />
+    <xacro:include filename="${t265_xacro_path}" />
+    <xacro:include filename="$(find omnibot_platform_description)/urdf/inertia_calc.xacro" />
     <!--  PLATFORM DESCRIPTION -->
+    <link name="base_footprint"></link>
     <link name="base_link">
         <inertial>
-            <origin xyz="${base_link_offset_x} ${base_link_offset_y} ${base_link_offset_z}"
-                rpy="${base_link_rotate_x} ${base_link_rotate_y} ${base_link_rotate_z}" />
+            <origin xyz="${base_link_offset_x} ${base_link_offset_y}
+        ${base_link_offset_z}"
+                rpy="${base_link_rotate_x} ${base_link_rotate_y}
+        ${base_link_rotate_z}" />
             <mass value="3.0" />
-            <inertia ixx="0.0" ixy="0.0" ixz="0.0" iyy="0.0" iyz="0.0" izz="0.0" />
+            <xacro:box_inertia m="3.0" x="${wheel_base_width}" y="${wheel_base_lenth}" z="0.2" />
         </inertial>
         <visual name="">
@@ -72,29 +95,52 @@
         </collision>
     </link>
+    <joint name="base_footprint_joint" type="fixed">
+        <parent link="base_footprint" />
+        <child link="base_link" />
+        <origin xyz="0.0 0.0 0.0" rpy="0.0 0.0 0.0" />
+    </joint>
     <xacro:mecanum_wheel name="left_front" side="1"
-        interface="hardware_interface/VelocityJointInterface">
+        interface="hardware_interface/VelocityJointInterface" parent="base_link">
         <origin xyz="${omniwheel_offset_x} ${omniwheel_offset_y} ${omniwheel_offset_z}"
             rpy="0.0 0.0 1.57" />
     </xacro:mecanum_wheel>
     <xacro:mecanum_wheel name="right_front" side="-1"
-        interface="hardware_interface/VelocityJointInterface">
+        interface="hardware_interface/VelocityJointInterface" parent="base_link">
         <origin xyz="${omniwheel_offset_x} ${-omniwheel_offset_y} ${omniwheel_offset_z}"
             rpy="0.0 0.0 1.57" />
     </xacro:mecanum_wheel>
     <xacro:mecanum_wheel name="left_back" side="-1"
-        interface="hardware_interface/VelocityJointInterface">
+        interface="hardware_interface/VelocityJointInterface" parent="base_link">
         <origin xyz="${-omniwheel_offset_x} ${omniwheel_offset_y} ${omniwheel_offset_z}"
             rpy="0.0 0.0 -1.57" />
     </xacro:mecanum_wheel>
     <xacro:mecanum_wheel name="right_back" side="1"
-        interface="hardware_interface/VelocityJointInterface">
+        interface="hardware_interface/VelocityJointInterface" parent="base_link">
         <origin xyz="${-omniwheel_offset_x} ${-omniwheel_offset_y} ${omniwheel_offset_z}"
             rpy="0.0 0.0 -1.57" />
     </xacro:mecanum_wheel>
-    <xacro:d435 offset_x="${0.196 + 0.0105+0.005}" offset_y="0.0" offset_z="0.114"
-        mesh_path="${rs_d435_mesh_path}" />
-    <xacro:realsense_T265 sensor_name="t265" parent_link="base_link" rate="30.0"
-        mesh_path="${rs_t265_mesh_path}">
-        <origin rpy="0 0 0" xyz="0.226500 0 0.094250" />
-    </xacro:realsense_T265>
+    <!-- <xacro:t265 sensor_name="t265" parent_link="base_link" rate="30.0"
+    mesh_path="${t265_mesh_path}">
+        <origin xyz="${t265_x_offset}  ${t265_y_offset} ${t265_z_offset}" rpy="0 0 0" />
+        <! <origin xyz="0.0 0.0 0.0" rpy="0.0 0.0 0.0"/> -->
+    <!-- </xacro:t265> -->
+    <!-- <xacro:d400
+    mesh_path="${d435_mesh_path}" parent_link="base_link">
+        <origin xyz="${d435_x_offset}
+    ${d435_y_offset}  ${d435_z_offset}" rpy="0.0 0.0 0.0" />
+    </xacro:d400> -->
+    <!-- <xacro:sensor_t265 parent="base_link" name="t265" topics_ns="t265">
+        <origin xyz="${t265_x_offset}  ${t265_y_offset} ${t265_z_offset}" rpy="0 0 0" />
+    </xacro:sensor_t265> -->
+    <!-- <xacro:sensor_d435 parent="t265_link" name="d400" topics_ns="d400"
+    use_nominal_extrinsics="true" add_plug="false" use_mesh="true" publish_pointcloud="true">
+        <origin xyz="${d435_x_offset} ${d435_y_offset}  ${d435_z_offset}" rpy="0.0 0.0 0.0" />
+    </xacro:sensor_d435> -->
+    <xacro:sensor_t265 parent="base_link" name="t265" topics_ns="t265"
+        odom_xyz="0.0 0.0 0.0" odom_rpy="0.0 0.0 0.0" unite_imu_method="true">
+        <origin xyz="${t265_x_offset}  ${t265_y_offset} ${t265_z_offset}" rpy="0 0 0" />
+    </xacro:sensor_t265>
+    <xacro:sensor_d435 parent="base_link" name="d400" topics_ns="d400" align_depth="true" enable_pointCloud="true">
+        <origin xyz="${d435_x_offset} ${d435_y_offset}  ${d435_z_offset}" rpy="0.0 0.0 0.0" />
+    </xacro:sensor_d435>
 </robot>
