Commit message: fix odom bugs, add sensor odom manager package

File: src/omnibot_platform/omnibot_platform_description/urdf/rollers.xacro (robot description, xacro)
@@ -1,25 +1,29 @@
-<?xml version="1.0" ?>
+<?xml version="1.0"?>
 <robot name="wheel" xmlns:xacro="http://www.ros.org/wiki/xacro">
-  <xacro:macro name="roller_origin" params="r th side wheel_side" >
+  <xacro:macro name="roller_origin" params="r th side wheel_side">
     <xacro:if value="${side==1 and wheel_side==1}">
-      <origin xyz="0 ${r*cos(th)} ${0.040289*sin(th)}" rpy="${atan(-tan(th)*sqrt(2.0))} ${asin(cos(th)/sqrt(2.0))} ${atan(sin(th))}"/>
+      <origin xyz="0 ${r*cos(th)} ${0.040289*sin(th)}"
+        rpy="${atan(-tan(th)*sqrt(2.0))} ${asin(cos(th)/sqrt(2.0))} ${atan(sin(th))}" />
     </xacro:if>
     <xacro:if value="${side==1 and wheel_side==-1}">
-      <origin xyz="0 ${r*cos(th)} ${0.040289*sin(th)}" rpy="${3.14+atan(-tan(th)*sqrt(2.0))} ${3.14+asin(cos(th)/sqrt(2.0))} ${atan(sin(th))}"/>
+      <origin xyz="0 ${r*cos(th)} ${0.040289*sin(th)}"
+        rpy="${3.14+atan(-tan(th)*sqrt(2.0))} ${3.14+asin(cos(th)/sqrt(2.0))} ${atan(sin(th))}" />
     </xacro:if>
     <xacro:if value="${side==-1 and wheel_side==1}">
-      <origin xyz="0 ${r*cos(th)} ${r*sin(th)}" rpy="${atan(-tan(th)*sqrt(2.0))} ${asin(-cos(th)/sqrt(2.0))} ${atan(-sin(th))}"/>
+      <origin xyz="0 ${r*cos(th)} ${r*sin(th)}"
+        rpy="${atan(-tan(th)*sqrt(2.0))} ${asin(-cos(th)/sqrt(2.0))} ${atan(-sin(th))}" />
     </xacro:if>
     <xacro:if value="${side==-1 and wheel_side==-1}">
-      <origin xyz="0 ${r*cos(th)} ${r*sin(th)}" rpy="${3.14+atan(-tan(th)*sqrt(2.0))} ${3.14+asin(-cos(th)/sqrt(2.0))} ${atan(-sin(th))}"/>
+      <origin xyz="0 ${r*cos(th)} ${r*sin(th)}"
+        rpy="${3.14+atan(-tan(th)*sqrt(2.0))} ${3.14+asin(-cos(th)/sqrt(2.0))} ${atan(-sin(th))}" />
     </xacro:if>
   </xacro:macro>
-  <xacro:macro name="roller_loop" params="name side num loop wheel_side2" >
+  <xacro:macro name="roller_loop" params="name side num loop wheel_side2">
     <xacro:if value="${loop}">
       <xacro:if value="${wheel_side2==1}">
-        <xacro:property name="joint_name" value="${name}_roller1_${loop}"/>
+        <xacro:property name="joint_name" value="${name}_roller_1_${loop}" />
       </xacro:if>
       <xacro:if value="${wheel_side2==-1}">
-        <xacro:property name="joint_name" value="${name}_roller2_${loop}"/>
+        <xacro:property name="joint_name" value="${name}_roller_2_${loop}" />
       </xacro:if>
       <link name="${joint_name}_link">
@@ -27,5 +31,6 @@
           <origin xyz="-0.002 0 0" rpy="0 0 0" />
           <geometry>
-            <mesh filename="package://omnibot_platform_description/meshes/wheel_roller2.dae" scale="0.001 0.001 0.001" />
+            <mesh filename="package://omnibot_platform_description/meshes/wheel_roller2.dae"
+              scale="0.001 0.001 0.001" />
           </geometry>
         </visual>
@@ -33,5 +38,6 @@
           <origin xyz="-0.002 0 0" rpy="0 0 0" />
           <geometry>
-            <mesh filename="package://omnibot_platform_description/meshes/wheel_roller2.dae" scale="0.001 0.001 0.001" />
+            <mesh filename="package://omnibot_platform_description/meshes/wheel_roller2.dae"
+              scale="0.001 0.001 0.001" />
           </geometry>
         </collision>
@@ -40,6 +46,6 @@
           <mass value="0.3" />
           <inertia ixx="0.00024000" ixy="0.0" ixz="0.0"
-                  iyy="0.00076000" iyz="0.0"
-                  izz="0.00076000" />
+            iyy="0.00076000" iyz="0.0"
+            izz="0.00076000" />
         </inertial>
         <surface>
@@ -64,8 +70,10 @@
       </link>
       <joint name="${joint_name}_joint" type="continuous">
-        <xacro:roller_origin th="${radians(360/num*(loop-1))}" side="${side}" wheel_side="${wheel_side2}" r="0.040293"/>
-        <axis xyz="1 0 0"/>
+        <xacro:roller_origin th="${radians(360/num*(loop-1))}" side="${side}"
+          wheel_side="${wheel_side2}" r="0.040293" />
+        <axis xyz="1 0 0" />
         <parent link="${name}_mecanum_wheel_link" />
         <child link="${joint_name}_link" />
+        <!-- <safety_controller k_velocity="10.0" /> -->
         <dynamics damping="0.001" friction="0.0001" />
       </joint>
@@ -80,15 +88,16 @@
         </actuator>
       </transmission>
-      <gazebo reference="${joint_name}_link">
-        <selfCollide>false</selfCollide>
-          <mu1 value="1.2" />
-          <mu2 value="1.2" />
-        </gazebo>
-      <xacro:roller_loop name="${name}" side="${side}" num="${num}" loop="${loop - 1}"  wheel_side2="${wheel_side2}"/>
+      <!-- <gazebo reference="${joint_name}_link">
+        <selfCollide>0</selfCollide>
+        <kp>1000000</kp>
+        <kd>100</kd>
+      </gazebo> -->
+      <xacro:roller_loop name="${name}" side="${side}" num="${num}" loop="${loop - 1}"
+        wheel_side2="${wheel_side2}" />
     </xacro:if>
   </xacro:macro>
   <xacro:macro name="rollers_link" params="name side">
-    <xacro:roller_loop name="${name}" side="${side}" num="7" loop="7" wheel_side2="1"/>
-    <xacro:roller_loop name="${name}" side="${side}" num="7" loop="7" wheel_side2="-1"/>
+    <xacro:roller_loop name="${name}" side="${side}" num="7" loop="7" wheel_side2="1" />
+    <xacro:roller_loop name="${name}" side="${side}" num="7" loop="7" wheel_side2="-1" />
   </xacro:macro>
 </robot>
