Commit message: commit for linux test

File: src/omnibot_platform/omnibot_platform_description/urdf/omnibot_platform.urdf.xacro (robot description, xacro)
@@ -1,70 +1,92 @@
 <?xml version="1.0"?>
 <robot xmlns:xacro="http://www.ros.org/wiki/xacro" name="omnibot_platform">
+    <gazebo>
+        <plugin name="gazebo_ros_control" filename="libgazebo_ros_control.so">
+            <robotNamespace>/</robotNamespace>
+        </plugin>
+    </gazebo>
     <!-- BASELINK  -->
-    <xacro:property name="wheel_base_width" value="0.306100"/>
-    <xacro:property name="wheel_base_lenth" value="0.336000"/>
-    <xacro:property name="base_link_offset_x" value="0.0"/>
-    <xacro:property name="base_link_offset_y" value="0.0"/>
-    <xacro:property name="base_link_offset_z" value="0.0"/>
-    <xacro:property name="base_link_rotate_x" value="0.0"/>
-    <xacro:property name="base_link_rotate_y" value="3.14"/>
-    <xacro:property name="base_link_rotate_z" value="-1.57"/>
-    <xacro:property name="base_link_mesh_path" value="package://omnibot_platform_description/meshes/base.dae"/>
-    <xacro:property name="base_link_mesh_scale_x" value="0.001"/>
-    <xacro:property name="base_link_mesh_scale_y" value="0.001"/>
-    <xacro:property name="base_link_mesh_scale_z" value="0.001"/>
+    <xacro:property name="wheel_base_width" value="0.306100" />
+    <xacro:property name="wheel_base_lenth" value="0.336000" />
+    <xacro:property name="base_link_offset_x" value="0.0" />
+    <xacro:property name="base_link_offset_y" value="0.0" />
+    <xacro:property name="base_link_offset_z" value="0.0" />
+    <xacro:property name="base_link_rotate_x" value="0.0" />
+    <xacro:property name="base_link_rotate_y" value="3.14" />
+    <xacro:property name="base_link_rotate_z" value="-1.57" />
+    <xacro:property name="base_link_mesh_path"
+        value="package://omnibot_platform_description/meshes/base.dae" />
+    <xacro:property name="base_link_mesh_scale_x" value="0.001" />
+    <xacro:property name="base_link_mesh_scale_y" value="0.001" />
+    <xacro:property name="base_link_mesh_scale_z" value="0.001" />
     <!-- OMNIWHEEL -->
-    <xacro:property name="omniwheel_offset_x" value="${(wheel_base_lenth / 2)}"/>
-    <xacro:property name="omniwheel_offset_y" value="${(wheel_base_width / 2)}"/>
-    <xacro:property name="omniwheel_offset_z" value="0.015500"/>
-    <xacro:property name="omniwheel_macro_path" value="$(find omnibot_platform_description)/urdf/omniwheel.urdf.xacro"/>
+    <xacro:property name="omniwheel_offset_x" value="${(wheel_base_lenth / 2)}" />
+    <xacro:property name="omniwheel_offset_y" value="${(wheel_base_width / 2)}" />
+    <xacro:property name="omniwheel_offset_z" value="0.015500" />
+    <xacro:property name="omniwheel_macro_path"
+        value="$(find omnibot_platform_description)/urdf/omniwheel.urdf.xacro" />
     <!-- REALSENSE -->
-    <xacro:property name="rs435_macro_path" value="$(find omnibot_platform_description)/urdf/d435.urdf.xacro"/>
-    <xacro:property name="rs265_macro_path" value="$(find omnibot_platform_description)/urdf/tracker.xacro"/>
-    <xacro:property name="rs_d435_mesh_path" value="package://omnibot_platform_description/meshes/d435.stl"/>
-    <xacro:property name="rs_t265_mesh_path" value="package://omnibot_platform_description/meshes/t265.stl"/>
+    <xacro:property name="rs435_macro_path"
+        value="$(find omnibot_platform_description)/urdf/d435.urdf.xacro" />
+    <xacro:property name="rs265_macro_path"
+        value="$(find omnibot_platform_description)/urdf/tracker.xacro" />
+    <xacro:property name="rs_d435_mesh_path"
+        value="package://omnibot_platform_description/meshes/d435.stl" />
+    <xacro:property name="rs_t265_mesh_path"
+        value="package://omnibot_platform_description/meshes/t265.stl" />
     <!--  INCLUDES -->
-    <xacro:include filename="${omniwheel_macro_path}"/>
-    <xacro:include filename="${rs435_macro_path}"/>
-    <xacro:include filename="${rs265_macro_path}"/>
+    <xacro:include filename="${omniwheel_macro_path}" />
+    <xacro:include filename="${rs435_macro_path}" />
+    <xacro:include filename="${rs265_macro_path}" />
     <!--  PLATFORM DESCRIPTION -->
     <link name="base_link">
         <inertial>
-            <origin xyz="${base_link_offset_x} ${base_link_offset_y} ${base_link_offset_z}" rpy="${base_link_rotate_x} ${base_link_rotate_y} ${base_link_rotate_z}"/>
-            <mass value="0.0"/>
-            <inertia ixx="0.0" ixy="0.0" ixz="0.0" iyy="0.0" iyz="0.0" izz="0.0"/>
+            <origin xyz="${base_link_offset_x} ${base_link_offset_y} ${base_link_offset_z}"
+                rpy="${base_link_rotate_x} ${base_link_rotate_y} ${base_link_rotate_z}" />
+            <mass value="3.0" />
+            <inertia ixx="0.0" ixy="0.0" ixz="0.0" iyy="0.0" iyz="0.0" izz="0.0" />
         </inertial>
         <visual name="">
-            <origin xyz="${base_link_offset_x} ${base_link_offset_y} ${base_link_offset_z}" rpy="${base_link_rotate_x} ${base_link_rotate_y} ${base_link_rotate_z}"/>
+            <origin xyz="${base_link_offset_x} ${base_link_offset_y} ${base_link_offset_z}"
+                rpy="${base_link_rotate_x} ${base_link_rotate_y} ${base_link_rotate_z}" />
             <geometry>
-                <mesh filename="${base_link_mesh_path}" scale="${base_link_mesh_scale_x} ${base_link_mesh_scale_y} ${base_link_mesh_scale_z}"/>
+                <mesh filename="${base_link_mesh_path}"
+                    scale="${base_link_mesh_scale_x} ${base_link_mesh_scale_y} ${base_link_mesh_scale_z}" />
             </geometry>
             <material name="">
-                <color rgba="1.0 0.0 0.0 1.0"/>
-                <texture filename=""/>
+                <color rgba="1.0 0.0 0.0 1.0" />
+                <texture filename="" />
             </material>
         </visual>
         <collision>
-            <origin xyz="${base_link_offset_x} ${base_link_offset_y} ${base_link_offset_z}" rpy="${base_link_rotate_x} ${base_link_rotate_y} ${base_link_rotate_z}"/>
+            <origin xyz="${base_link_offset_x} ${base_link_offset_y} ${base_link_offset_z}"
+                rpy="${base_link_rotate_x} ${base_link_rotate_y} ${base_link_rotate_z}" />
             <geometry>
-                <mesh filename="${base_link_mesh_path}" scale="${base_link_mesh_scale_x} ${base_link_mesh_scale_y} ${base_link_mesh_scale_z}"/>
+                <mesh filename="${base_link_mesh_path}"
+                    scale="${base_link_mesh_scale_x} ${base_link_mesh_scale_y} ${base_link_mesh_scale_z}" />
             </geometry>
         </collision>
     </link>
-    <xacro:omniwheel_macro suffix="left_forward">
-        <origin xyz="${omniwheel_offset_x} ${omniwheel_offset_y} ${omniwheel_offset_z}" rpy="0.0 0.0 0.0"/>
+    <xacro:omniwheel_macro suffix="left_front">
+        <origin xyz="${omniwheel_offset_x} ${omniwheel_offset_y} ${omniwheel_offset_z}"
+            rpy="0.0 0.0 0.0" />
     </xacro:omniwheel_macro>
-    <xacro:omniwheel_macro suffix="right_forward">
-        <origin xyz="${omniwheel_offset_x} ${-omniwheel_offset_y} ${omniwheel_offset_z}" rpy="0.0 0.0 3.14"/>
+    <xacro:omniwheel_macro suffix="right_front">
+        <origin xyz="${omniwheel_offset_x} ${-omniwheel_offset_y} ${omniwheel_offset_z}"
+            rpy="0.0 0.0 3.14" />
     </xacro:omniwheel_macro>
-    <xacro:omniwheel_macro suffix="left_backward">
-        <origin xyz="${-omniwheel_offset_x} ${omniwheel_offset_y} ${omniwheel_offset_z}" rpy="0.0 0.0 0.0"/>
+    <xacro:omniwheel_macro suffix="left_back">
+        <origin xyz="${-omniwheel_offset_x} ${omniwheel_offset_y} ${omniwheel_offset_z}"
+            rpy="0.0 0.0 0.0" />
     </xacro:omniwheel_macro>
-    <xacro:omniwheel_macro suffix="right_backward">
-        <origin xyz="${-omniwheel_offset_x} ${-omniwheel_offset_y} ${omniwheel_offset_z}" rpy="0.0 0.0 3.14"/>
+    <xacro:omniwheel_macro suffix="right_back">
+        <origin xyz="${-omniwheel_offset_x} ${-omniwheel_offset_y} ${omniwheel_offset_z}"
+            rpy="0.0 0.0 3.14" />
     </xacro:omniwheel_macro>
-    <xacro:d435 offset_x="${0.196 + 0.0105}" offset_y="0.0" offset_z="0.114" mesh_path="${rs_d435_mesh_path}"/>
-    <xacro:realsense_T265 sensor_name="t265" parent_link="base_link" rate="30.0" mesh_path="${rs_t265_mesh_path}">
-        <origin rpy="0 0 0" xyz="0.226500 0 0.094250"/>
+    <xacro:d435 offset_x="${0.196 + 0.0105}" offset_y="0.0" offset_z="0.114"
+        mesh_path="${rs_d435_mesh_path}" />
+    <xacro:realsense_T265 sensor_name="t265" parent_link="base_link" rate="30.0"
+        mesh_path="${rs_t265_mesh_path}">
+        <origin rpy="0 0 0" xyz="0.226500 0 0.094250" />
     </xacro:realsense_T265>
 </robot>

File: src/omnibot_platform/omnibot_platform_description/urdf/omniwheel.urdf.xacro (robot description, xacro)
@@ -1,39 +1,64 @@
 <?xml version="1.0"?>
 <robot xmlns:xacro="http://www.ros.org/wiki/xacro" name="omniwheel">
-    <xacro:property name="omniwheel_mesh_path" value="package://omnibot_platform_description/meshes/wheel.dae"/>
-    <xacro:property name="omniwheel_mesh_scale_x" value="0.001"/>
-    <xacro:property name="omniwheel_mesh_scale_y" value="0.001"/>
-    <xacro:property name="omniwheel_mesh_scale_z" value="0.001"/>
+    <xacro:include filename="$(find omnibot_platform_description)/urdf/inertia_calc.xacro"/>
+    <xacro:property name="omniwheel_mesh_path"
+        value="package://omnibot_platform_description/meshes/wheel.dae" />
+    <xacro:property name="omniwheel_mesh_scale_x" value="0.001" />
+    <xacro:property name="omniwheel_mesh_scale_y" value="0.001" />
+    <xacro:property name="omniwheel_mesh_scale_z" value="0.001" />
+    <xacro:property name="omniwheel_mass" value="0.5" />
+    <xacro:property name="omniwheel_deameter" value="0.15" />
+    <xacro:property name="omniwheel_radius" value="${omniwheel_deameter/2}" />
+    <xacro:property name="omniwheel_width" value="0.3" />
     <xacro:macro name="omniwheel_macro" params="suffix *origin">
-        <joint name="${suffix}_wheel_joint" type="revolute">
-            <xacro:insert_block name="origin"/>
-            <parent link="base_link"/>
-            <child link="${suffix}_omniwheel_link"/>
-            <axis xyz="0 1 0"/>
-            <limit lower="-3.14" upper="3.14" effort="1000.0" velocity="50.0"/>
-        </joint>
         <link name="${suffix}_omniwheel_link">
             <inertial>
-                <origin xyz="0.0 0.0 0.0" rpy="0.0 0.0 0.0"/>
-                <mass value="0.0"/>
-                <inertia ixx="0.0" ixy="0.0" ixz="0.0" iyy="0.0" iyz="0.0" izz="0.0"/>
+                <origin xyz="0.0 0.0 0.0" rpy="0.0 0.0 0.0" />
+                <mass value="${omniwheel_mass}" />
+                <!-- <inertia ixx="0.0" ixy="0.0" ixz="0.0" iyy="0.0" iyz="0.0" izz="0.0" /> -->
+                <xacro:cylinder_inertia m="${omniwheel_mass}" r="${omniwheel_radius}" h="${omniwheel_width}"></xacro:cylinder_inertia>
             </inertial>
             <visual name="">
-                <origin xyz="0.0 0.0 0.0" rpy="0.0 0.0 0.0"/>
+                <origin xyz="0.0 0.0 0.0" rpy="0.0 0.0 0.0" />
                 <geometry>
-                    <mesh filename="${omniwheel_mesh_path}" scale="${omniwheel_mesh_scale_x} ${omniwheel_mesh_scale_y} ${omniwheel_mesh_scale_z}"/>
+                    <mesh filename="${omniwheel_mesh_path}"
+                        scale="${omniwheel_mesh_scale_x} ${omniwheel_mesh_scale_y} ${omniwheel_mesh_scale_z}" />
                 </geometry>
                 <material name="">
-                    <color rgba="1.0 0.0 0.0 1.0"/>
-                    <texture filename=""/>
+                    <color rgba="1.0 0.0 0.0 1.0" />
+                    <texture filename="" />
                 </material>
             </visual>
             <collision>
-            <origin xyz="0.0 0.0 0.0" rpy="0.0 0.0 0.0"/>
+                <origin xyz="0.0 0.0 0.0" rpy="0.0 0.0 0.0" />
                 <geometry>
-                    <mesh filename="${omniwheel_mesh_path}" scale="${omniwheel_mesh_scale_x} ${omniwheel_mesh_scale_y} ${omniwheel_mesh_scale_z}"/>
+                    <mesh filename="${omniwheel_mesh_path}"
+                        scale="${omniwheel_mesh_scale_x} ${omniwheel_mesh_scale_y} ${omniwheel_mesh_scale_z}" />
                 </geometry>
             </collision>
         </link>
+        <transmission name="${suffix}_omniwheel_trans">
+            <type>transmission_interface/SimpleTransmission</type>
+            <actuator name="${suffix}_omniwheel_motor">
+                <mechanicalReduction>1</mechanicalReduction>
+            </actuator>
+            <joint name="${suffix}_omniwheel_joint">
+                <hardwareInterface>hardware_interface/VelocityJointInterface</hardwareInterface>
+            </joint>
+        </transmission>
+        <joint name="${suffix}_omniwheel_joint" type="revolute">
+            <xacro:insert_block name="origin" />
+            <parent link="base_link" />
+            <child link="${suffix}_omniwheel_link" />
+            <axis xyz="0 1 0" />
+            <limit lower="-3.14" upper="3.14" effort="1000.0" velocity="50.0" />
+        </joint>
+        <gazebo reference="${suffix}_omniwheel">
+            <mu1 value="200.0" />
+            <mu2 value="100.0" />
+            <kp value="10000000.0" />
+            <kd value="1.0" />
+            <material>Gazebo/Grey</material>
+        </gazebo>
     </xacro:macro>
 </robot>

Commit message: change mecanum wheel model

File: src/omnibot_platform/omnibot_platform_description/urdf/omnibot_platform.urdf.xacro (robot description, xacro)
@@ -22,8 +22,12 @@
     <!-- OMNIWHEEL -->
     <xacro:property name="omniwheel_offset_x" value="${(wheel_base_lenth / 2)}" />
-    <xacro:property name="omniwheel_offset_y" value="${(wheel_base_width / 2)}" />
+    <xacro:property name="omniwheel_offset_y" value="${(wheel_base_width / 2) + 0.035}" />
     <xacro:property name="omniwheel_offset_z" value="0.015500" />
+    <!--
     <xacro:property name="omniwheel_macro_path"
-        value="$(find omnibot_platform_description)/urdf/omniwheel.urdf.xacro" />
+            value="$(find
+    omnibot_platform_description)/urdf/omniwheel.urdf.xacro" /> -->
+    <xacro:property name="omniwheel_macro_path"
+        value="$(find omnibot_platform_description)/urdf/mecanum_wheel_macro.xacro" />
     <!-- REALSENSE -->
     <xacro:property name="rs435_macro_path"
@@ -68,20 +72,45 @@
         </collision>
     </link>
-    <xacro:omniwheel_macro suffix="left_front">
-        <origin xyz="${omniwheel_offset_x} ${omniwheel_offset_y} ${omniwheel_offset_z}"
+    <!-- <xacro:omniwheel_macro suffix="left_front">
+        <origin xyz="${omniwheel_offset_x}
+    ${omniwheel_offset_y} ${omniwheel_offset_z}"
             rpy="0.0 0.0 0.0" />
     </xacro:omniwheel_macro>
     <xacro:omniwheel_macro suffix="right_front">
-        <origin xyz="${omniwheel_offset_x} ${-omniwheel_offset_y} ${omniwheel_offset_z}"
-            rpy="0.0 0.0 3.14" />
+        <origin
+    xyz="${omniwheel_offset_x} ${-omniwheel_offset_y} ${omniwheel_offset_z}"
+            rpy="0.0
+    0.0 3.14" />
     </xacro:omniwheel_macro>
     <xacro:omniwheel_macro suffix="left_back">
-        <origin xyz="${-omniwheel_offset_x} ${omniwheel_offset_y} ${omniwheel_offset_z}"
-            rpy="0.0 0.0 0.0" />
+    <origin xyz="${-omniwheel_offset_x} ${omniwheel_offset_y} ${omniwheel_offset_z}"
+            rpy="0.0
+    0.0 0.0" />
     </xacro:omniwheel_macro>
     <xacro:omniwheel_macro suffix="right_back">
+    <origin xyz="${-omniwheel_offset_x} ${-omniwheel_offset_y} ${omniwheel_offset_z}"
+            rpy="0.0
+    0.0 3.14" />
+    </xacro:omniwheel_macro> -->
+    <xacro:mecanum_wheel name="left_front" side="1"
+        interface="hardware_interface/EffortJointInterface">
+        <origin xyz="${omniwheel_offset_x} ${omniwheel_offset_y} ${omniwheel_offset_z}"
+            rpy="0.0 0.0 1.57" />
+    </xacro:mecanum_wheel>
+    <xacro:mecanum_wheel name="right_front" side="-1"
+        interface="hardware_interface/EffortJointInterface">
+        <origin xyz="${omniwheel_offset_x} ${-omniwheel_offset_y} ${omniwheel_offset_z}"
+            rpy="0.0 0.0 1.57" />
+    </xacro:mecanum_wheel>
+    <xacro:mecanum_wheel name="left_back" side="-1"
+        interface="hardware_interface/EffortJointInterface">
+        <origin xyz="${-omniwheel_offset_x} ${omniwheel_offset_y} ${omniwheel_offset_z}"
+            rpy="0.0 0.0 -1.57" />
+    </xacro:mecanum_wheel>
+    <xacro:mecanum_wheel name="right_back" side="1"
+        interface="hardware_interface/EffortJointInterface">
         <origin xyz="${-omniwheel_offset_x} ${-omniwheel_offset_y} ${omniwheel_offset_z}"
-            rpy="0.0 0.0 3.14" />
-    </xacro:omniwheel_macro>
+            rpy="0.0 0.0 -1.57" />
+    </xacro:mecanum_wheel>
     <xacro:d435 offset_x="${0.196 + 0.0105+0.005}" offset_y="0.0" offset_z="0.114"
         mesh_path="${rs_d435_mesh_path}" />

Commit message: add occupancy pkg

File: src/omnibot_platform/omnibot_platform_description/urdf/omnibot_platform.urdf.xacro (robot description, xacro)
@@ -72,25 +72,4 @@
         </collision>
     </link>
-    <!-- <xacro:omniwheel_macro suffix="left_front">
-        <origin xyz="${omniwheel_offset_x}
-    ${omniwheel_offset_y} ${omniwheel_offset_z}"
-            rpy="0.0 0.0 0.0" />
-    </xacro:omniwheel_macro>
-    <xacro:omniwheel_macro suffix="right_front">
-        <origin
-    xyz="${omniwheel_offset_x} ${-omniwheel_offset_y} ${omniwheel_offset_z}"
-            rpy="0.0
-    0.0 3.14" />
-    </xacro:omniwheel_macro>
-    <xacro:omniwheel_macro suffix="left_back">
-    <origin xyz="${-omniwheel_offset_x} ${omniwheel_offset_y} ${omniwheel_offset_z}"
-            rpy="0.0
-    0.0 0.0" />
-    </xacro:omniwheel_macro>
-    <xacro:omniwheel_macro suffix="right_back">
-    <origin xyz="${-omniwheel_offset_x} ${-omniwheel_offset_y} ${omniwheel_offset_z}"
-            rpy="0.0
-    0.0 3.14" />
-    </xacro:omniwheel_macro> -->
     <xacro:mecanum_wheel name="left_front" side="1"
         interface="hardware_interface/VelocityJointInterface">

Commit message: combine manipulator and platform packages

File: src/omnibot_platform/omnibot_platform_description/urdf/omnibot_platform.urdf.xacro (robot description, xacro)
@@ -3,16 +3,7 @@
     <gazebo>
         <plugin name="gazebo_ros_control" filename="libgazebo_ros_control.so">
-            <robotNamespace>/</robotNamespace>
+            <robotNamespace>/omnibot_platform</robotNamespace>
         </plugin>
     </gazebo>
-    <!-- <gazebo>
-        <plugin name="object_controller" filename="libgazebo_ros_planar_move.so">
-    <commandTopic>cmd_vel</commandTopic>
-            <odometryTopic>odom</odometryTopic>
-    <odometryFrame>odom</odometryFrame>
-            <odometryRate>20.0</odometryRate>
-    <robotBaseFrame>base_link</robotBaseFrame>
-        </plugin>
-    </gazebo> -->
     <!-- BASELINK  -->
     <xacro:property name="wheel_base_width" value="0.306100" />
@@ -36,6 +27,5 @@
         value="$(find omnibot_platform_description)/urdf/mecanum_wheel_macro.xacro" />
     <!-- REALSENSE -->
-<!--
-    <xacro:property name="t265_xacro_path"
+    <!-- <xacro:property name="t265_xacro_path"
         value="$(find omnibot_platform_description)/urdf/t265.xacro" />
     <xacro:property name="t265_mesh_path"
@@ -64,5 +54,5 @@
     <xacro:include filename="$(find omnibot_platform_description)/urdf/inertia_calc.xacro" />
     <!--  PLATFORM DESCRIPTION -->
-    <link name="base_footprint"></link>
+    <link name="base_footprint"/>
     <link name="base_link">
         <inertial>
@@ -120,21 +110,4 @@
             rpy="0.0 0.0 -1.57" />
     </xacro:mecanum_wheel>
-    <!-- <xacro:t265 sensor_name="t265" parent_link="base_link" rate="30.0"
-    mesh_path="${t265_mesh_path}">
-        <origin xyz="${t265_x_offset}  ${t265_y_offset} ${t265_z_offset}" rpy="0 0 0" />
-        <! <origin xyz="0.0 0.0 0.0" rpy="0.0 0.0 0.0"/> -->
-    <!-- </xacro:t265> -->
-    <!-- <xacro:d400
-    mesh_path="${d435_mesh_path}" parent_link="base_link">
-        <origin xyz="${d435_x_offset}
-    ${d435_y_offset}  ${d435_z_offset}" rpy="0.0 0.0 0.0" />
-    </xacro:d400> -->
-    <!-- <xacro:sensor_t265 parent="base_link" name="t265" topics_ns="t265">
-        <origin xyz="${t265_x_offset}  ${t265_y_offset} ${t265_z_offset}" rpy="0 0 0" />
-    </xacro:sensor_t265> -->
-    <!-- <xacro:sensor_d435 parent="t265_link" name="d400" topics_ns="d400"
-    use_nominal_extrinsics="true" add_plug="false" use_mesh="true" publish_pointcloud="true">
-        <origin xyz="${d435_x_offset} ${d435_y_offset}  ${d435_z_offset}" rpy="0.0 0.0 0.0" />
-    </xacro:sensor_d435> -->
     <xacro:sensor_t265 parent="base_link" name="t265" topics_ns="t265"
         odom_xyz="0.0 0.0 0.0" odom_rpy="0.0 0.0 0.0" unite_imu_method="true">
