Commit message: add slamtech rplidar A3 3d-model  and urdf model

File: src/omnibot_platform/omnibot_platform_description/urdf/omnibot_platform.urdf.xacro (robot description, xacro)
@@ -31,29 +31,34 @@
         value="$(find omnibot_platform_description)/urdf/mecanum_wheel_macro.xacro" />
     <!-- REALSENSE -->
-    <!-- <xacro:property name="t265_xacro_path"
-        value="$(find omnibot_platform_description)/urdf/t265.xacro" />
-    <xacro:property name="t265_mesh_path"
-        value="package://omnibot_platform_description/meshes/t265.stl" /> -->
     <xacro:property name="t265_xacro_path"
         value="$(find omnibot_platform_description)/urdf/_t265.urdf.xacro" />
+    <xacro:property name="d435_xacro_path"
+        value="$(find omnibot_platform_description)/urdf/_d435.urdf.xacro" />
     <xacro:property name="t265_x_offset" value="0.226500" />
     <xacro:property name="t265_y_offset" value="0.0" />
     <xacro:property name="t265_z_offset" value="0.094250" />
-    <!-- <xacro:property name="d435_xacro_path"
-        value="$(find omnibot_platform_description)/urdf/d435.urdf.xacro" />
-    <xacro:property name="d435_mesh_path"
-        value="package://omnibot_platform_description/meshes/d435.stl" /> -->
-    <xacro:property name="d435_xacro_path"
-        value="$(find omnibot_platform_description)/urdf/_d435.urdf.xacro" />
+    <xacro:property name="t265_x_rotate" value="0.0" />
+    <xacro:property name="t265_y_rotate" value="0.0" />
+    <xacro:property name="t265_z_rotate" value="0.0" />
     <xacro:property name="d435_x_offset" value="${0.196 + 0.0105 + 0.005}" />
     <xacro:property name="d435_y_offset" value="0.0" />
     <xacro:property name="d435_z_offset" value="0.114" />
-    <!-- <xacro:property name="d435_x_offset" value="-0.01950" />
-    <xacro:property name="d435_y_offset" value="0.0" />
-    <xacro:property name="d435_z_offset" value="0.019" /> -->
+    <xacro:property name="d435_x_rotate" value="0.0" />
+    <xacro:property name="d435_y_rotate" value="0.0" />
+    <xacro:property name="d435_z_rotate" value="0.0" />
+    <!-- LIDAR -->
+    <xacro:property name="rplidar_a3_xacro_path"
+        value="$(find omnibot_platform_description)/urdf/rplidar_a3.urdf.xacro" />
+    <xacro:property name="rplidar_a3_x_offset" value="0.00"/>
+    <xacro:property name="rplidar_a3_y_offset" value="0.00"/>
+    <xacro:property name="rplidar_a3_z_offset" value="0.00"/>
+    <xacro:property name="rplidar_a3_x_rotate" value="0.00"/>
+    <xacro:property name="rplidar_a3_y_rotate" value="0.00"/>
+    <xacro:property name="rplidar_a3_z_rotate" value="0.00"/>
     <!--  INCLUDES -->
     <xacro:include filename="${omniwheel_macro_path}" />
     <xacro:include filename="${d435_xacro_path}" />
     <xacro:include filename="${t265_xacro_path}" />
+    <xacro:include filename="${rplidar_a3_xacro_path}"/>
     <xacro:include filename="$(find omnibot_platform_description)/urdf/inertia_calc.xacro" />
     <!--  PLATFORM DESCRIPTION -->
@@ -121,3 +126,7 @@
         <origin xyz="${d435_x_offset} ${d435_y_offset}  ${d435_z_offset}" rpy="0.0 0.0 0.0" />
     </xacro:sensor_d435>
+    <xacro:rplidar_a3 suffix="front">
+        <origin xyz="0.0 0.0 0.0" rpy="0.0 0.0 0.0"/>
+        <parent link="base_link"/>
+    </xacro:rplidar_a3>
 </robot>

File: src/omnibot_platform/omnibot_platform_description/urdf/rplidar_a3.urdf.xacro (robot description, xacro)
@@ -42,5 +42,5 @@
                 <origin xyz="0.0 0.0 0.0" rpy="0.0 0.0 0.0" />
                 <geometry>
-                    <mesh filename="package://acar_description/meshes/rplidar-a2m4-r1.STL" scale="0.001 0.001 0.001"/>
+                    <mesh filename="package://omnibot_platform_description/meshes/rplidarA3.dae" scale="0.001 0.001 0.001"/>
                 </geometry>
                 <material name="">
@@ -52,5 +52,5 @@
                 <origin xyz="0.0 0.0 0.0" rpy="0.0 0.0 0.0" />
                 <geometry>
-                    <mesh filename="package://acar_description/meshes/rplidar-a2m4-r1.STL" scale="0.001 0.001 0.001"/>
+                    <mesh filename="package://omnibot_platform_description/meshes/rplidarA3.dae" scale="0.001 0.001 0.001"/>
                 </geometry>
             </collision>

Commit message: fix platform descr

File: src/omnibot_platform/omnibot_platform_description/urdf/omnibot_platform.urdf.xacro (robot description, xacro)
@@ -15,5 +15,5 @@
     <xacro:property name="base_link_offset_x" value="0.0" />
     <xacro:property name="base_link_offset_y" value="0.0" />
-    <xacro:property name="base_link_offset_z" value="0.00" />
+    <xacro:property name="base_link_offset_z" value="0.0" />
     <xacro:property name="base_link_rotate_x" value="0.0" />
     <xacro:property name="base_link_rotate_y" value="3.14" />
@@ -35,13 +35,13 @@
     <xacro:property name="d435_xacro_path"
         value="$(find omnibot_platform_description)/urdf/_d435.urdf.xacro" />
-    <xacro:property name="t265_x_offset" value="0.226500" />
+    <xacro:property name="t265_x_offset" value="${0.191250 + 0.0135}" />
     <xacro:property name="t265_y_offset" value="0.0" />
-    <xacro:property name="t265_z_offset" value="0.094250" />
+    <xacro:property name="t265_z_offset" value="${0.202950 - 0.035}" />
     <xacro:property name="t265_x_rotate" value="0.0" />
     <xacro:property name="t265_y_rotate" value="0.0" />
     <xacro:property name="t265_z_rotate" value="0.0" />
-    <xacro:property name="d435_x_offset" value="${0.196 + 0.0105 + 0.005}" />
+    <xacro:property name="d435_x_offset" value="${0.176250 + 0.012}" />
     <xacro:property name="d435_y_offset" value="0.0" />
-    <xacro:property name="d435_z_offset" value="0.114" />
+    <xacro:property name="d435_z_offset" value="${0.230460 - 0.05}" />
     <xacro:property name="d435_x_rotate" value="0.0" />
     <xacro:property name="d435_y_rotate" value="0.0" />
@@ -50,10 +50,10 @@
     <xacro:property name="rplidar_a3_xacro_path"
         value="$(find omnibot_platform_description)/urdf/rplidar_a3.urdf.xacro" />
-    <xacro:property name="rplidar_a3_x_offset" value="0.00"/>
-    <xacro:property name="rplidar_a3_y_offset" value="0.00"/>
-    <xacro:property name="rplidar_a3_z_offset" value="0.00"/>
+    <xacro:property name="rplidar_a3_x_offset" value="0.168000"/>
+    <xacro:property name="rplidar_a3_y_offset" value="0.0"/>
+    <xacro:property name="rplidar_a3_z_offset" value="${0.148960 - 0.035}"/>
     <xacro:property name="rplidar_a3_x_rotate" value="0.00"/>
     <xacro:property name="rplidar_a3_y_rotate" value="0.00"/>
-    <xacro:property name="rplidar_a3_z_rotate" value="0.00"/>
+    <xacro:property name="rplidar_a3_z_rotate" value="1.57"/>
     <!--  INCLUDES -->
     <xacro:include filename="${omniwheel_macro_path}" />
@@ -97,5 +97,5 @@
         <parent link="base_footprint" />
         <child link="base_link" />
-        <origin xyz="0.0 0.0 0.08" rpy="0.0 0.0 0.0" />
+        <origin xyz="0.0 0.0 0.03" rpy="0.0 0.0 0.0" />
     </joint>
     <xacro:mecanum_wheel name="left_front" side="1"
@@ -121,11 +121,11 @@
     <xacro:sensor_t265 parent="base_link" name="t265" topics_ns="t265"
         odom_xyz="0.0 0.0 0.0" odom_rpy="0.0 0.0 0.0" unite_imu_method="true">
-        <origin xyz="${t265_x_offset}  ${t265_y_offset} ${t265_z_offset}" rpy="0 0 0" />
+        <origin xyz="${t265_x_offset}  ${t265_y_offset} ${t265_z_offset}" rpy="${t265_x_rotate}  ${t265_y_rotate} ${t265_z_rotate}" />
     </xacro:sensor_t265>
-    <xacro:sensor_d435 parent="base_link" name="d400" topics_ns="d400" align_depth="true" enable_pointCloud="true">
-        <origin xyz="${d435_x_offset} ${d435_y_offset}  ${d435_z_offset}" rpy="0.0 0.0 0.0" />
+    <xacro:sensor_d435 parent="base_link" name="d435" topics_ns="d435" align_depth="true" enable_pointCloud="true">
+        <origin xyz="${d435_x_offset} ${d435_y_offset}  ${d435_z_offset}" rpy="${d435_x_rotate} ${d435_y_rotate}  ${d435_z_rotate}" />
     </xacro:sensor_d435>
     <xacro:rplidar_a3 suffix="front">
-        <origin xyz="0.0 0.0 0.0" rpy="0.0 0.0 0.0"/>
+        <origin xyz="${rplidar_a3_x_offset} ${rplidar_a3_y_offset} ${rplidar_a3_z_offset}" rpy="${rplidar_a3_x_rotate} ${rplidar_a3_y_rotate} ${rplidar_a3_z_rotate}"/>
         <parent link="base_link"/>
     </xacro:rplidar_a3>

Commit message: add gazebo package launch file, setup bringup launch file ro sim, add worlds

File: src/omnibot_platform/omnibot_platform_description/urdf/omnibot_platform.urdf.xacro (robot description, xacro)
@@ -20,5 +20,5 @@
     <xacro:property name="base_link_rotate_z" value="-1.57" />
     <xacro:property name="base_link_mesh_path"
-        value="package://omnibot_platform_description/meshes/ros_base_link.dae" />
+        value="file://$(find omnibot_platform_description)/meshes/ros_base_link.dae" />
     <xacro:property name="base_link_mesh_scale_x" value="0.001" />
     <xacro:property name="base_link_mesh_scale_y" value="0.001" />
@@ -119,5 +119,5 @@
             rpy="0.0 0.0 -1.57" />
     </xacro:mecanum_wheel>
-    <xacro:sensor_t265 parent="base_link" name="t265" topics_ns="t265"
+    <!-- <xacro:sensor_t265 parent="base_link" name="t265" topics_ns="t265"
         odom_xyz="0.0 0.0 0.0" odom_rpy="0.0 0.0 0.0" unite_imu_method="true">
         <origin xyz="${t265_x_offset}  ${t265_y_offset} ${t265_z_offset}" rpy="${t265_x_rotate}  ${t265_y_rotate} ${t265_z_rotate}" />
@@ -125,5 +125,5 @@
     <xacro:sensor_d435 parent="base_link" name="d435" topics_ns="d435" align_depth="true" enable_pointCloud="true">
         <origin xyz="${d435_x_offset} ${d435_y_offset}  ${d435_z_offset}" rpy="${d435_x_rotate} ${d435_y_rotate}  ${d435_z_rotate}" />
-    </xacro:sensor_d435>
+    </xacro:sensor_d435> -->
     <xacro:rplidar_a3 suffix="front">
         <origin xyz="${rplidar_a3_x_offset} ${rplidar_a3_y_offset} ${rplidar_a3_z_offset}" rpy="${rplidar_a3_x_rotate} ${rplidar_a3_y_rotate} ${rplidar_a3_z_rotate}"/>

File: src/omnibot_platform/omnibot_platform_description/urdf/rollers.xacro (robot description, xacro)
@@ -31,5 +31,5 @@
           <origin xyz="-0.002 0 0" rpy="0 0 0" />
           <geometry>
-            <mesh filename="package://omnibot_platform_description/meshes/wheel_roller2.dae"
+            <mesh filename="file://$(find omnibot_platform_description)/meshes/wheel_roller2.dae"
               scale="0.001 0.001 0.001" />
           </geometry>
@@ -38,5 +38,5 @@
           <origin xyz="-0.002 0 0" rpy="0 0 0" />
           <geometry>
-            <mesh filename="package://omnibot_platform_description/meshes/wheel_roller2.dae"
+            <mesh filename="file://$(find omnibot_platform_description)/meshes/wheel_roller2.dae"
               scale="0.001 0.001 0.001" />
           </geometry>

File: src/omnibot_platform/omnibot_platform_description/urdf/rplidar_a3.urdf.xacro (robot description, xacro)
@@ -42,5 +42,5 @@
                 <origin xyz="0.0 0.0 0.0" rpy="0.0 0.0 0.0" />
                 <geometry>
-                    <mesh filename="package://omnibot_platform_description/meshes/rplidarA3.dae" scale="0.001 0.001 0.001"/>
+                    <mesh filename="file://$(find omnibot_platform_description)/meshes/rplidarA3.dae" scale="0.001 0.001 0.001"/>
                 </geometry>
                 <material name="">
@@ -52,5 +52,5 @@
                 <origin xyz="0.0 0.0 0.0" rpy="0.0 0.0 0.0" />
                 <geometry>
-                    <mesh filename="package://omnibot_platform_description/meshes/rplidarA3.dae" scale="0.001 0.001 0.001"/>
+                    <mesh filename="file://$(find omnibot_platform_description)/meshes/rplidarA3.dae" scale="0.001 0.001 0.001"/>
                 </geometry>
             </collision>

File: src/omnibot_platform/omnibot_platform_description/urdf/wheel.xacro (robot description, xacro)
@@ -6,5 +6,5 @@
         <origin xyz="0 0 0" rpy="0 0 ${1.57 * side}" />
         <geometry>
-          <mesh filename="package://omnibot_platform_description/meshes/wheel_base.dae" scale="${side / 1000} 0.001 0.001" />
+          <mesh filename="file://$(find omnibot_platform_description)/meshes/wheel_base.dae" scale="${side / 1000} 0.001 0.001" />
         </geometry>
       </visual>
@@ -12,5 +12,5 @@
         <origin xyz="0 0 0" rpy="0 0 ${1.57 * side}" />
         <geometry>
-          <mesh filename="package://omnibot_platform_description/meshes/wheel_base.dae" scale="${side / 1000} 0.001 0.001" />
+          <mesh filename="file://$(find omnibot_platform_description)/meshes/wheel_base.dae" scale="${side / 1000} 0.001 0.001" />
         </geometry>
       </collision>
@@ -30,5 +30,5 @@
         <origin xyz="0 0.035 0" rpy="0 0 ${1.57 * side}" />
         <geometry>
-          <mesh filename="package://omnibot_platform_description/meshes/adapter.dae" scale="${side / 1000} 0.001 0.001" />
+          <mesh filename="file://$(find omnibot_platform_description)/meshes/adapter.dae" scale="${side / 1000} 0.001 0.001" />
         </geometry>
       </visual>
@@ -36,5 +36,5 @@
         <origin xyz="0 0.035 0" rpy="0 0 ${1.57 * side}" />
         <geometry>
-          <mesh filename="package://omnibot_platform_description/meshes/adapter.dae" scale="${side / 1000} 0.001 0.001" />
+          <mesh filename="file://$(find omnibot_platform_description)/meshes/adapter.dae" scale="${side / 1000} 0.001 0.001" />
         </geometry>
       </collision>
