Commit message: add lidar

File: src/omnibot_platform/omnibot_platform_description/urdf/rplidar_a3.urdf.xacro (robot description, xacro)
@@ -2,6 +2,65 @@
 <robot xmlns:xacro="http://www.ros.org/wiki/xacro" name="rplidar_a3">
     <xacro:macro name="rplidar_a3" params="suffix *origin *parent">
-        <gazebo reference="laser">
-            <sensor type="gpu_ray" name="head_rplidar_sensor">
+        <link name="${suffix}_rplidar_a3_link">
+            <inertial>
+                <origin xyz="0.0 0.0 0.0" rpy="0.0 0.0 0.0" />
+                <mass value="0.0" />
+                <inertia ixx="0.0" ixy="0.0" ixz="0.0" iyy="0.0" iyz="0.0" izz="0.0" />
+            </inertial>
+            <visual name="">
+                <origin xyz="0.0 0.0 0.0" rpy="0.0 0.0 0.0" />
+                <geometry>
+                    <mesh filename="file://$(find omnibot_platform_description)/meshes/rplidarA3.dae" scale="0.001 0.001 0.001"/>
+                </geometry>
+            </visual>
+            <collision>
+                <origin xyz="0.0 0.0 0.0" rpy="0.0 0.0 0.0" />
+                <geometry>
+                    <mesh filename="file://$(find omnibot_platform_description)/meshes/rplidarA3.dae" scale="0.001 0.001 0.001"/>
+                </geometry>
+            </collision>
+        </link>
+        <joint name="${suffix}_rplidar_a3_joint" type="fixed">
+            <xacro:insert_block name="parent"/>
+            <child link="${suffix}_rplidar_a3_link"/>
+            <xacro:insert_block name="origin"/>
+        </joint>
+         <gazebo reference="${suffix}_rplidar_a3_link">
+            <sensor name="${suffix}_lidar_sensor" type="gpu_lidar">
+                <gz_frame_id>${suffix}_rplidar_a3_link</gz_frame_id>
+                <topic>scan</topic>
+                <update_rate>40</update_rate>
+                                <always_on>true</always_on>
+                <visualize>true</visualize>
+                <ray>
+                    <scan>
+                        <horizontal>
+                            <samples>720</samples>
+                            <resolution>1</resolution>
+                            <min_angle>-3.14159265</min_angle>
+                            <max_angle>3.14159265</max_angle>
+                        </horizontal>
+                        <vertical>
+                            <samples>1</samples>
+                            <resolution>1</resolution>
+                            <min_angle>0</min_angle>
+                            <max_angle>0</max_angle>
+                        </vertical>
+                    </scan>
+                    <range>
+                        <min>0.2</min>
+                        <max>25.0</max>
+                        <resolution>0.01</resolution>
+                    </range>
+                    <noise>
+                        <type>gaussian</type>
+                        <mean>0.0</mean>
+                        <stddev>0.01</stddev>
+                    </noise>
+                </ray>
+            </sensor>
+        </gazebo>
+    </xacro:macro>
+ <!-- <sensor type="gpu_lidar" name="head_rplidar_sensor">
                 <pose>0 0 0.06 0 0 0</pose>
                 <visualize>true</visualize>
@@ -31,30 +90,4 @@
                     <frameName>laser</frameName>
                 </plugin>
-            </sensor>
-        </gazebo>
-        <link name="${suffix}_rplidar_a3_link">
-            <inertial>
-                <origin xyz="0.0 0.0 0.0" rpy="0.0 0.0 0.0" />
-                <mass value="0.0" />
-                <inertia ixx="0.0" ixy="0.0" ixz="0.0" iyy="0.0" iyz="0.0" izz="0.0" />
-            </inertial>
-            <visual name="">
-                <origin xyz="0.0 0.0 0.0" rpy="0.0 0.0 0.0" />
-                <geometry>
-                    <mesh filename="file://$(find omnibot_platform_description)/meshes/rplidarA3.dae" scale="0.001 0.001 0.001"/>
-                </geometry>
-            </visual>
-            <collision>
-                <origin xyz="0.0 0.0 0.0" rpy="0.0 0.0 0.0" />
-                <geometry>
-                    <mesh filename="file://$(find omnibot_platform_description)/meshes/rplidarA3.dae" scale="0.001 0.001 0.001"/>
-                </geometry>
-            </collision>
-        </link>
-        <joint name="${suffix}_rplidar_a3_joint" type="fixed">
-            <xacro:insert_block name="parent"/>
-            <child link="${suffix}_rplidar_a3_link"/>
-            <xacro:insert_block name="origin"/>
-        </joint>
-    </xacro:macro>
+            </sensor> -->
 </robot>
