Commit message: add start comdition for gz_sim

File: src/omnibot_platform/omnibot_platform_description/urdf/omnibot_platform_description.urdf.xacro (robot description, xacro)
@@ -42,8 +42,4 @@
                     scale="${base_link_mesh_scale_x} ${base_link_mesh_scale_y} ${base_link_mesh_scale_z}" />
             </geometry>
-            <material name="">
-                <color rgba="1.0 0.0 0.0 1.0" />
-                <texture filename="" />
-            </material>
         </visual>
         <collision>

Commit message: add worlds, fix lidar "xray"

File: src/omnibot_platform/omnibot_platform_description/urdf/omnibot_platform_description.urdf.xacro (robot description, xacro)
@@ -5,5 +5,13 @@
         <plugin filename="gz_ros2_control-system" name="gz_ros2_control::GazeboSimROS2ControlPlugin">
             <parameters>$(find omnibot_platform_control)/config/omnibot_platform_ros2_controllers.yaml</parameters>
+            <ros>
+                <remapping>/controller_manager/robot_description:=/robot_description</remapping>
+            </ros>
         </plugin>
+        <!-- <plugin
+            filename="gz-sim-sensors-system"
+            name="gz::sim::systems::Sensors">
+            <render_engine>ogre2</render_engine>
+        </plugin> -->
     </gazebo>
     <ros2_control name="OmnibotPlatformSystem" type="system">
@@ -111,5 +119,5 @@
     <!-- BASE_LINK -->
     <xacro:property name="base_link_mesh_path"
-        value="file://$(find omnibot_platform_description)/meshes/base_link.dae" />
+        value="file://$(find omnibot_platform_description)/meshes/omnibot_base_link.dae" />
     <xacro:property name="base_link_offset_x" value="0.0" />
     <xacro:property name="base_link_offset_y" value="0.0" />
@@ -168,4 +176,14 @@
         </collision>
     </link>
+    <gazebo reference="base_link">
+    <material>
+            <ambient>0.1 0.1 0.1 1</ambient>
+            <diffuse>0.1 0.1 0.1 1</diffuse>
+            <specular>0.1 0.1 0.1 1</specular>
+    </material>
+        <visibility_flags>1</visibility_flags>
+        <self_collide>0</self_collide>
+        <kinematic>1</kinematic>
+    </gazebo>
     <joint name="base_footprint_joint" type="fixed">
         <parent link="base_footprint" />

File: src/omnibot_platform/omnibot_platform_description/urdf/rplidar_a3.urdf.xacro (robot description, xacro)
@@ -1,5 +1,9 @@
 <?xml version="1.0"?>
 <robot xmlns:xacro="http://www.ros.org/wiki/xacro" name="rplidar_a3">
-    <xacro:macro name="rplidar_a3" params="suffix *origin *parent">
+    <xacro:macro name="rplidar_a3"
+        params="suffix *origin *parent
+    gazebo_material_ambient:='0.1 0.1 0.1 1'
+    gazebo_material_diffuse:='0.1 0.1 0.1 1'
+    gazebo_material_specular:='0.1 0.1 0.1 1'">
         <link name="${suffix}_rplidar_a3_link">
             <inertial>
@@ -11,5 +15,7 @@
                 <origin xyz="0.0 0.0 0.0" rpy="0.0 0.0 0.0" />
                 <geometry>
-                    <mesh filename="file://$(find omnibot_platform_description)/meshes/rplidarA3.dae" scale="0.001 0.001 0.001"/>
+                    <mesh
+                        filename="file://$(find omnibot_platform_description)/meshes/rplidarA3.dae"
+                        scale="0.001 0.001 0.001" />
                 </geometry>
             </visual>
@@ -17,27 +23,39 @@
                 <origin xyz="0.0 0.0 0.0" rpy="0.0 0.0 0.0" />
                 <geometry>
-                    <mesh filename="file://$(find omnibot_platform_description)/meshes/rplidarA3.dae" scale="0.001 0.001 0.001"/>
+                    <mesh
+                        filename="file://$(find omnibot_platform_description)/meshes/rplidarA3.dae"
+                        scale="0.001 0.001 0.001" />
                 </geometry>
             </collision>
         </link>
         <joint name="${suffix}_rplidar_a3_joint" type="fixed">
-            <xacro:insert_block name="parent"/>
-            <child link="${suffix}_rplidar_a3_link"/>
-            <xacro:insert_block name="origin"/>
+            <xacro:insert_block name="parent" />
+            <child link="${suffix}_rplidar_a3_link" />
+            <xacro:insert_block name="origin" />
         </joint>
-         <gazebo reference="${suffix}_rplidar_a3_link">
+        <link name="${suffix}_rplidar_a3_scan_link" />
+        <joint name="${suffix}_rplidar_a3_scan_joint" type="fixed">
+            <parent link="${suffix}_rplidar_a3_link" />
+            <child link="${suffix}_rplidar_a3_scan_link" />
+            <origin xyz="0.0 0.0 0.03" rpy="0.0 0.0 0.0" />
+        </joint>
+        <gazebo reference="${suffix}_rplidar_a3_scan_link">
+            <material>
+                <ambient>${gazebo_material_ambient}</ambient>
+                <diffuse>${gazebo_material_diffuse}</diffuse>
+                <specular>${gazebo_material_specular}</specular>
+            </material>
             <sensor name="${suffix}_lidar_sensor" type="gpu_lidar">
-                <gz_frame_id>${suffix}_rplidar_a3_link</gz_frame_id>
                 <topic>scan</topic>
                 <update_rate>40</update_rate>
-                                <always_on>true</always_on>
+                <always_on>true</always_on>
                 <visualize>true</visualize>
-                <ray>
+                <lidar>
                     <scan>
                         <horizontal>
                             <samples>720</samples>
                             <resolution>1</resolution>
-                            <min_angle>-3.14159265</min_angle>
-                            <max_angle>3.14159265</max_angle>
+                            <min_angle>-3.1415</min_angle>
+                            <max_angle>3.1415</max_angle>
                         </horizontal>
                         <vertical>
@@ -49,5 +67,5 @@
                     </scan>
                     <range>
-                        <min>0.2</min>
+                        <min>0.0385</min>
                         <max>25.0</max>
                         <resolution>0.01</resolution>
@@ -58,9 +76,12 @@
                         <stddev>0.01</stddev>
                     </noise>
-                </ray>
+                    <visibility_mask>4294967294</visibility_mask>
+                    <frame_id>${suffix}_rplidar_a3_scan_link</frame_id>
+                </lidar>
+                <gz_frame_id>${suffix}_rplidar_a3_scan_link</gz_frame_id>
             </sensor>
         </gazebo>
     </xacro:macro>
- <!-- <sensor type="gpu_lidar" name="head_rplidar_sensor">
+    <!-- <sensor type="gpu_lidar" name="head_rplidar_sensor">
                 <pose>0 0 0.06 0 0 0</pose>
                 <visualize>true</visualize>

Commit message: add mecanum driver

File: src/omnibot_platform/omnibot_platform_description/urdf/omnibot_platform_description.urdf.xacro (robot description, xacro)
@@ -136,5 +136,5 @@
     <xacro:property name="wheel_offset_y" value="${(wheel_base_width / 2) + 0.035}" />
     <xacro:property name="wheel_offset_z" value="0.015500" />
-    <!-- LIDAR -->
+    <!-- RPLIDAR A3 -->
     <xacro:property name="rplidar_a3_xacro_path" value="rplidar_a3.urdf.xacro" />
     <xacro:property name="rplidar_a3_x_offset" value="0.168000" />
@@ -144,7 +144,16 @@
     <xacro:property name="rplidar_a3_y_rotate" value="0.00" />
     <xacro:property name="rplidar_a3_z_rotate" value="1.57" />
+    <!-- REALSENSE D435 -->
+    <xacro:property name="d435_x_offset" value="${0.176250 + 0.012}" />
+    <xacro:property name="d435_y_offset" value="0.0" />
+    <xacro:property name="d435_z_offset" value="${0.230460 - 0.05}" />
+    <xacro:property name="d435_x_rotate" value="0.0" />
+    <xacro:property name="d435_y_rotate" value="0.0" />
+    <xacro:property name="d435_z_rotate" value="0.0" />
+    <xacro:property name="d435_xacro_path"
+        value="$(find omnibot_platform_description)/urdf/_d435.urdf.xacro" />
     <!--  INCLUDES -->
     <xacro:include filename="${wheel_macro_path}" />
-    <!-- <xacro:include filename="${d435_xacro_path}" /> -->
+    <xacro:include filename="${d435_xacro_path}" />
     <!-- <xacro:include filename="${t265_xacro_path}" /> -->
     <xacro:include filename="${rplidar_a3_xacro_path}" />
@@ -177,9 +186,9 @@
     </link>
     <gazebo reference="base_link">
-    <material>
+        <material>
             <ambient>0.1 0.1 0.1 1</ambient>
             <diffuse>0.1 0.1 0.1 1</diffuse>
             <specular>0.1 0.1 0.1 1</specular>
-    </material>
+        </material>
         <visibility_flags>1</visibility_flags>
         <self_collide>0</self_collide>
@@ -216,3 +225,6 @@
         <parent link="base_link" />
     </xacro:rplidar_a3>
+    <xacro:sensor_d435 parent_link="base_link" name="d435" topics_ns="d435" align_depth="true" publish_pointcloud="true">
+        <origin xyz="${d435_x_offset} ${d435_y_offset}  ${d435_z_offset}" rpy="0.0 0.0 0.0" />
+    </xacro:sensor_d435>
 </robot>
