File: electronic/jetson_power_board/untitled.sch (EAGLE design)
At the start: 20 parts

Commit message: add sim models
Parts:
- added LED2: (no value), led:LED5MM
- added R6: (no value), resistor:R-EU_R0805
- C10, C9: device resistor:CPOL-EU153CLV-0405 -> resistor:CPOL-EU153CLV-0810
Connections:
- new net N$5: LED2.C, R6.1
- net GND: now also R6.2
- net VDD: now also LED2.A

Commit message: some model changes
Parts:
- removed D1: CGRM4004-G, diode:CGRM4004-G
- removed LED1: (no value), led:LEDCHIPLED_0805
- removed LED2: (no value), led:LED5MM
- removed R3, R4, R5, R6: (no value), resistor:R-EU_R0805
- added C11: (no value), resistor:CPOL-EU153CLV-0810
- added J3: (no value), SparkFun-Connectors:CONN_025MM
- added U1: (no value), SparkFun-IC-Power:V_REG_LM1117SOT223
Connections:
- removed net N$3: D1.C, LED1.A, R3.1, R4.1, U$1.EN
- removed net N$4: LED1.C, R5.1
- net GND: now also C11.-, J3.2, U1.ADJ; no longer D1.A, R4.2, R5.2, R6.2
- net N$5: now also C11.+, J3.1, U1.OUT, U1.OUT@1; no longer LED2.C, R6.1
- net V+: no longer R3.2
- net VDD: now also U1.IN; no longer LED2.A
