File: electronic/low_level_contoller_board/low_level_contoller_board.brd (EAGLE design)
At the start: 97.5 x 57.1 mm, 11 parts

Commit message: some model changes
Parts:
- removed J6: (no value), SparkFun-Connectors:1X04
Connections:
- removed net N$15: J6.3, U$1.10
- removed net N$16: J6.2, U$1.13
- net +3V3: no longer J6.4
- net GND: no longer J6.1
Routing:
- net N$15: track 49.5 -> 0.00 mm
- net N$16: track 39.4 -> 0.00 mm
- net GND: track 218.4 -> 182.3 mm
- net +3V3: track 226.6 -> 221.5 mm
Changed lines of the file:
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@@
 <drawing>
 <settings>
-<setting alwaysvectorfont="yes"/>
+<setting alwaysvectorfont="no"/>
 <setting verticaltext="up"/>
 </settings>
@@
 <attribute name="PROD_ID" value="CONN-09696" x="96.52" y="66.04" size="1.778" layer="27" rot="R270" display="off"/>
 </element>
-<element name="J6" library="SparkFun-Connectors" package="1X04" value="" x="96.52" y="21.59" rot="R90">
-<attribute name="PROD_ID" value="CONN-09696" x="96.52" y="21.59" size="1.778" layer="27" rot="R90" display="off"/>
-</element>
 <element name="J7" library="SparkFun-Connectors" package="1X04" value="" x="69.85" y="25.4" rot="R180">
 <attribute name="PROD_ID" value="CONN-09696" x="69.85" y="25.4" size="1.778" layer="27" rot="R180" display="off"/>
@@
 <wire x1="6.35" y1="24.13" x2="39.37" y2="24.13" width="1.27" layer="16"/>
 </signal>
-<signal name="N$15">
-<contactref element="U$1" pad="10"/>
-<contactref element="J6" pad="3"/>
-<wire x1="62.23" y1="31.75" x2="62.23" y2="36.83" width="1.27" layer="16"/>
-<wire x1="87.63" y1="36.83" x2="62.23" y2="36.83" width="1.27" layer="16"/>
-<wire x1="96.52" y1="26.67" x2="87.63" y2="26.67" width="1.27" layer="16"/>
-<wire x1="87.63" y1="26.67" x2="87.63" y2="36.83" width="1.27" layer="16"/>
-</signal>
-<signal name="N$16">
-<contactref element="J6" pad="2"/>
-<contactref element="U$1" pad="13"/>
-<wire x1="69.85" y1="31.75" x2="69.85" y2="34.29" width="1.27" layer="16"/>
-<wire x1="85.09" y1="34.29" x2="69.85" y2="34.29" width="1.27" layer="16"/>
-<wire x1="96.52" y1="24.13" x2="85.09" y2="24.13" width="1.27" layer="16"/>
-<wire x1="85.09" y1="24.13" x2="85.09" y2="34.29" width="1.27" layer="16"/>
-</signal>
 <signal name="GND">
 <contactref element="J4" pad="1"/>
-<contactref element="J6" pad="1"/>
 <wire x1="6.35" y1="21.59" x2="62.23" y2="21.59" width="1.27" layer="16"/>
 <contactref element="J3" pad="1"/>
 <contactref element="J5" pad="4"/>
-<wire x1="62.23" y1="21.59" x2="96.52" y2="21.59" width="1.27" layer="16"/>
 <wire x1="4.191" y1="21.59" x2="6.35" y2="21.59" width="1.27" layer="16"/>
-<wire x1="96.52" y1="21.59" x2="98.349" y2="21.59" width="1.27" layer="16"/>
 <wire x1="98.349" y1="21.59" x2="98.349" y2="58.42" width="1.27" layer="16"/>
 <wire x1="98.349" y1="58.42" x2="96.52" y2="58.42" width="1.27" layer="16"/>
@@
 <wire x1="34.29" y1="31.75" x2="34.29" y2="35.56" width="1.27" layer="16"/>
 <wire x1="34.29" y1="35.56" x2="4.191" y2="35.56" width="1.27" layer="16"/>
+<wire x1="62.23" y1="21.59" x2="98.349" y2="21.59" width="0" layer="19" extent="16-16"/>
 </signal>
 <signal name="+3V3">
 <contactref element="J4" pad="4"/>
-<contactref element="J6" pad="4"/>
 <contactref element="J5" pad="1"/>
 <contactref element="J3" pad="4"/>
@@
 <wire x1="69.85" y1="25.4" x2="69.85" y2="27.94" width="1.27" layer="16"/>
 <wire x1="92.71" y1="66.04" x2="92.71" y2="54.61" width="1.27" layer="1"/>
-<wire x1="96.52" y1="29.21" x2="91.44" y2="29.21" width="1.27" layer="16"/>
 <wire x1="91.44" y1="29.21" x2="91.44" y2="36.83" width="1.27" layer="16"/>
 <contactref element="U$1" pad="3.3V"/>
