File: electronic/low_level_contoller_board/low_level_contoller_board.sch (EAGLE design)
At the start: 11 parts

Commit message: some model changes
Parts:
- removed J6: (no value), SparkFun-Connectors:CONN_04
Connections:
- removed net N$15: J6.3, U$1.10
- removed net N$16: J6.2, U$1.13
- net +3V3: no longer J6.4
- net GND: no longer J6.1
