Commit message: fix worlds bug

File: src/omnibot_manipulator/omnibot_manipulator_description/urdf/omnibot_manipulator.urdf.xacro (robot description, xacro)
@@ -221,4 +221,10 @@
 		</collision>
 	</link>
+	<link name="tip_link"/>
+	<joint name="tip_joint" type="fixed">
+		<parent link="ang_link5"/>
+		<child link="tip_link"/>
+		<origin xyz="0.0 0.0 -0.1" rpy="0.0 0.0 0.0"/>
+	</joint>
 	<joint name="ang_gripper" type="prismatic">
 		<parent link="ang_link5" />

File: src/omnibot_manipulator/omnibot_manipulator_moveit/config/gazebo_omnibot_robot.urdf (robot description, URDF)
Before this commit: robot omnibot_robot, 94 links, 93 joints
Links:
- added link tip_link
Joints:
- added joint tip_joint: type fixed, parent ang_link5, child tip_link, origin xyz=0.0 0.0 -0.1 rpy=0.0 0.0 0.0

Commit message: add firmware V3, change planners params

File: src/omnibot_manipulator/omnibot_manipulator_description/urdf/omnibot_manipulator.urdf.xacro (robot description, xacro)
@@ -225,5 +225,5 @@
 		<parent link="ang_link5"/>
 		<child link="tip_link"/>
-		<origin xyz="0.0 0.0 -0.1" rpy="0.0 0.0 0.0"/>
+		<origin xyz="0.0 0.0 -0.118" rpy="0.0 0.0 0.0"/>
 	</joint>
 	<joint name="ang_gripper" type="prismatic">

File: src/omnibot_manipulator/omnibot_manipulator_moveit/config/gazebo_omnibot_robot.urdf (robot description, URDF)
Before this commit: robot omnibot_robot, 95 links, 94 joints
Joints:
- joint tip_joint: origin xyz=0.0 0.0 -0.1 rpy=0.0 0.0 0.0 -> xyz=0.0 0.0 -0.118 rpy=0.0 0.0 0.0

Commit message: att d435 to manipulator

File: src/omnibot_manipulator/omnibot_manipulator_description/urdf/omnibot_manipulator.urdf.xacro (robot description, xacro)
@@ -11,4 +11,13 @@
 		</gazebo>
 	</xacro:unless>
+	<xacro:property name="d435_xacro_path"
+		value="$(find realsense_gazebo_description)/urdf/_d435.urdf.xacro" />
+    <xacro:include filename="${d435_xacro_path}" />
+	<xacro:property name="d435_x_offset" value="0.04" />
+	<xacro:property name="d435_y_offset" value="0.0" />
+	<xacro:property name="d435_z_offset" value="-0.023" />
+	<xacro:property name="d435_x_rotate" value="0.0" />
+	<xacro:property name="d435_y_rotate" value="1.57" />
+	<xacro:property name="d435_z_rotate" value="0.0" />
 	<xacro:include
 		filename="$(find omnibot_manipulator_description)/urdf/omnibot_manipulator.gazebo" />
@@ -221,9 +230,9 @@
 		</collision>
 	</link>
-	<link name="tip_link"/>
+	<link name="tip_link" />
 	<joint name="tip_joint" type="fixed">
-		<parent link="ang_link5"/>
-		<child link="tip_link"/>
-		<origin xyz="0.0 0.0 -0.118" rpy="0.0 0.0 0.0"/>
+		<parent link="ang_link5" />
+		<child link="tip_link" />
+		<origin xyz="0.0 0.0 -0.118" rpy="0.0 0.0 0.0" />
 	</joint>
 	<joint name="ang_gripper" type="prismatic">
@@ -288,3 +297,7 @@
 		</inertial>
 	</link>
+	<xacro:sensor_d435 parent="ang_link5" name="d400_arm" topics_ns="d400_arm" align_depth="true"
+		enable_pointCloud="true">
+		<origin xyz="${d435_x_offset} ${d435_y_offset}  ${d435_z_offset}" rpy="${d435_x_rotate} ${d435_y_rotate} ${d435_z_rotate}" />
+	</xacro:sensor_d435>
 </robot>
