Commit message: real manipulator works with moveit

File: src/omnibot_manipulator/omnibot_manipulator_moveit/config/gazebo_omnibot_robot.urdf (robot description, URDF)
Before this commit: robot omnibot_robot, 95 links, 94 joints
Links:
- added link d400_arm_bottom_screw_frame
- added link d400_arm_color_frame
- added link d400_arm_color_optical_frame
- added link d400_arm_depth_frame
- added link d400_arm_depth_optical_frame
- added link d400_arm_left_ir_frame
- added link d400_arm_left_ir_optical_frame
- added link d400_arm_link, mass 0.564; collision box size=0.02505 0.09 0.025; visual mesh filename=package://realsense2_description/meshes/d435.dae
- added link d400_arm_right_ir_frame
- added link d400_arm_right_ir_optical_frame
Joints:
- added joint d400_arm_color_joint: type fixed, parent d400_arm_depth_frame, child d400_arm_color_frame, origin xyz=0 0.015 0 rpy=0 0 0
- added joint d400_arm_color_optical_joint: type fixed, parent d400_arm_color_frame, child d400_arm_color_optical_frame, origin xyz=0 0 0 rpy=-1.5707963267948966 0 -1.5707963267948966
- added joint d400_arm_depth_joint: type fixed, parent d400_arm_link, child d400_arm_depth_frame, origin xyz=0 0 0 rpy=0 0 0
- added joint d400_arm_depth_optical_joint: type fixed, parent d400_arm_depth_frame, child d400_arm_depth_optical_frame, origin xyz=0 0 0 rpy=-1.5707963267948966 0 -1.5707963267948966
- added joint d400_arm_joint: type fixed, parent ang_link5, child d400_arm_bottom_screw_frame, origin xyz=0.04 0.0  -0.023 rpy=0.0 1.57 0.0
- added joint d400_arm_left_ir_joint: type fixed, parent d400_arm_depth_frame, child d400_arm_left_ir_frame, origin xyz=0 0.0 0 rpy=0 0 0
- added joint d400_arm_left_ir_optical_joint: type fixed, parent d400_arm_left_ir_frame, child d400_arm_left_ir_optical_frame, origin xyz=0 0 0 rpy=-1.5707963267948966 0 -1.5707963267948966
- added joint d400_arm_link_joint: type fixed, parent d400_arm_bottom_screw_frame, child d400_arm_link, origin xyz=0 0.0175 0.0125 rpy=0 0 0
- added joint d400_arm_right_ir_joint: type fixed, parent d400_arm_depth_frame, child d400_arm_right_ir_frame, origin xyz=0 -0.05 0 rpy=0 0 0
- added joint d400_arm_right_ir_optical_joint: type fixed, parent d400_arm_right_ir_frame, child d400_arm_right_ir_optical_frame, origin xyz=0 0 0 rpy=-1.5707963267948966 0 -1.5707963267948966
