File: electronic/BATTERIES_CONTROLLER _V3/BATTERIES_CONTROLLER _V3.sch (EAGLE design)
At the start: 17 parts, among them K1 FRS1B

Commit message: some changes
Parts:
- removed D1: 1N4004, diode:1N4004
- removed K1: FRS1B, relay:FRS1B
- R10, R11, R12, R13, R2, R3: value (none) -> 10k
- R14, R15, R16, R6, R7, R9: value (none) -> 100k
Connections:
- net N$18 renamed RX
- net N$19 renamed TX
- net N$20 renamed +5V
- removed net GND: D1.A, J3.1, K11.2, K12.O, K12.P, K12.P@1, R10.2, R11.2, R12.2, R13.2, R2.2, R3.2, U$1.GND, U$1.GND2
- removed net GNDA: J1.3, J1.5, J1.6, J1.7, K12.S
- removed net N$8: D1.C, K11.1, U$1.D10
- new net N$1: J1.3, J1.5, J1.6, J1.7, R10.2, R11.2, R12.2, R13.2, R2.2, R3.2
- new net N$4: U$1.GND
- new net N$5: J3.1, U$1.GND2
Other:
- moved on the sheet: R10, R11, R12, R14, R15, R16, R6, R7
